Commit message: feat: v00 urdf fix

File: lv2_module6/urdf/beebot_normal/urdf.xacro (robot description, xacro)
@@ -1,275 +1,544 @@
-<?xml version="1.0"?>
+<?xml version="1.0" ?>
 <!--
-  beebot — TurtleBot3 Waffle Pi + 앞쪽 상판(한 단) 위 매니퓰레이터(OM-X + 손목 roll + 그리퍼) + 뒤쪽 전원선 가이드 폴 (더미 치수)
+  beebot — 실측 CAD(bee.urdf, SolidWorks 내보내기)에서 만든 모델. bee.urdf를 새로 받으면 이 파일을 다시 만든다:
+    · 메시 경로: meshes/x.stl → meshes/x.stl
+    · 이름 맞춤(제어·시뮬레이터가 쓰는 이름): camera_rear → front_pole_cam, camera_wrist → gripper_cam,
+      gripper_joint → gripper_left_joint, gripper_mimic_joint → gripper_right_joint, tcp → end_effector
+    · 추가: imu_link · <ros2_control> 블록(BeebotSystemHardware) · xacro 인자
   설계: documents/ros2-design/07-tf.md (TF 트리), 08-ctrl.md (ros2_control)
   좌표: base_footprint(바닥) → base_link(바퀴 축 아래 0.010m), x 앞 · y 왼쪽 · z 위
-    - 차체: Waffle Pi 본체 266×266mm, 바퀴 반경 0.033m · 간격 0.287m, 뒤쪽 캐스터 2개
-    - 상판(deck): 차체 위 앞쪽 절반만 덮는 판넬, 스탠드오프 0.05m 위
-    - 매니퓰레이터: 상판 위 OpenMANIPULATOR-X + 손목 roll — 구동 관절 6개
-        joint1 yaw · joint2~4 pitch (OM-X) · joint5 손목 roll (추가) · gripper_left_joint (평행 그리퍼)
-    - 선가이드 폴: 차체 위 뒤쪽 끝, 전원선이 위에서 내려온다. pole_cam은 이 폴 위에 전방 하향으로 단다 (가정)
-    - gripper_cam: 그리퍼 몸체(gripper_link) 위에 얹은 RealSense
+  구동 관절 6개: joint1~5 (팔) · gripper_left_joint (평행 그리퍼, 0=닫힘 · 0.0265=열림, 오른쪽은 mimic) + 바퀴 2개
   xacro 인자:
     mock_hardware (false)  true면 control/BeebotSystemHardware가 실기 대신 명령을 그대로 상태로 되돌려 줌 (테스트베드)
     mock_effort   (0.0)    mock일 때 팔 관절 effort[A] (arm_safety_monitor 시험용)
     port          (/dev/opencr)  OpenCR 포트 (udev 고정 이름 — ros2_ws/99-opencr.rules)
-  TODO(권형중): 실측 치수·질량, 메시 (OM-X는 ROBOTIS open_manipulator_description/meshes STL을 쓸 수 있음), 손목 roll 모듈 실제 길이
-  Isaac Sim용 USD는 이 파일을 xacro로 펼친 URDF를 Isaac Sim URDF Importer로 변환해 만든다:
-    xacro beebot.urdf.xacro > beebot.urdf
 -->
+<!-- generated by make_xacro.py -->
 <robot name="beebot" xmlns:xacro="http://www.ros.org/wiki/xacro">
   <xacro:arg name="mock_hardware" default="false"/>
   <xacro:arg name="mock_effort" default="0.0"/>
   <xacro:arg name="port" default="/dev/opencr"/>
-  <xacro:property name="PI" value="3.14159265"/>
-  <!-- 차체 -->
-  <xacro:property name="wheel_radius" value="0.033"/>
-  <xacro:property name="wheel_width" value="0.018"/>
-  <xacro:property name="wheel_separation" value="0.287"/>
-  <xacro:property name="body_l" value="0.266"/>
-  <xacro:property name="body_w" value="0.266"/>
-  <xacro:property name="body_h" value="0.110"/>
-  <xacro:property name="body_x" value="-0.064"/>   <!-- 바퀴 축 기준 본체 중심 (바퀴가 앞쪽) -->
-  <xacro:property name="body_z" value="0.080"/>
-  <xacro:property name="body_top" value="${body_z + body_h / 2}"/>
-  <!-- 상판: 본체 앞쪽 절반 -->
-  <xacro:property name="deck_standoff" value="0.050"/>
-  <xacro:property name="deck_t" value="0.005"/>
-  <xacro:property name="deck_l" value="${body_l / 2}"/>
-  <xacro:property name="deck_x" value="${body_x + body_l / 4}"/>
-  <xacro:property name="deck_top" value="${body_top + deck_standoff + deck_t}"/>
-  <!-- 선가이드 폴: 본체 뒤쪽 끝 -->
-  <xacro:property name="pole_h" value="0.450"/>
-  <xacro:property name="pole_r" value="0.010"/>
-  <xacro:property name="pole_x" value="${body_x - body_l / 2 + 0.020}"/>
-  <material name="dark"><color rgba="0.2 0.2 0.2 1"/></material>
-  <material name="grey"><color rgba="0.6 0.6 0.6 1"/></material>
-  <material name="white"><color rgba="0.95 0.95 0.95 1"/></material>
-  <material name="orange"><color rgba="0.95 0.5 0.1 1"/></material>
-  <material name="blue"><color rgba="0.2 0.4 0.8 1"/></material>
-  <!-- 관성: 균질 직육면체·원기둥·구 -->
-  <xacro:macro name="box_inertia" params="m x y z *origin">
-    <inertial>
-      <xacro:insert_block name="origin"/>
-      <mass value="${m}"/>
-      <inertia ixx="${m * (y*y + z*z) / 12}" ixy="0" ixz="0" iyy="${m * (x*x + z*z) / 12}" iyz="0" izz="${m * (x*x + y*y) / 12}"/>
-    </inertial>
-  </xacro:macro>
-  <xacro:macro name="cylinder_inertia" params="m r h *origin">
-    <inertial>
-      <xacro:insert_block name="origin"/>
-      <mass value="${m}"/>
-      <inertia ixx="${m * (3*r*r + h*h) / 12}" ixy="0" ixz="0" iyy="${m * (3*r*r + h*h) / 12}" iyz="0" izz="${m * r * r / 2}"/>
-    </inertial>
-  </xacro:macro>
-  <!-- ================= 베이스 =================
-       링크·관절 이름과 TF 트리는 beebot_mesh/urdf.xacro와 같다 (모델을 바꿔 끼워도 노드·설정이 그대로 돎).
-       beebot_mesh처럼 차체에 붙은 것(캐스터·상판·적재함·선가이드 폴)은 base_link 한 링크의 도형으로 합쳤다. -->
-  <!-- 적재함 (뒤쪽 절반, 퍽 운반): 바닥 윗면 z=0.140 (base_link 기준) · 가이드벽 4면 (높이 0.04, 두께 0.005)
-       시뮬레이터는 같은 치수로 퍽 받침·가둠 판정 (simulator/main.py TRAY) -->
-  <xacro:property name="tray_x0" value="-0.19"/>
-  <xacro:property name="tray_x1" value="-0.07"/>
-  <xacro:property name="tray_y" value="0.10"/>
-  <xacro:property name="tray_floor_z" value="0.140"/>
-  <xacro:property name="tray_wall_h" value="0.04"/>
-  <xacro:property name="tray_wall_t" value="0.005"/>
-  <xacro:macro name="part" params="xyz *geometry material">
-    <visual>
-      <origin xyz="${xyz}"/>
-      <xacro:insert_block name="geometry"/>
-      <material name="${material}"/>
-    </visual>
-  </xacro:macro>
+  <xacro:arg name="mesh_uri" default="package://ros_system/urdf/meshes"/>
   <link name="base_footprint"/>
-  <link name="base_link">
-    <!-- 본체 -->
-    <visual>
-      <origin xyz="${body_x} 0 ${body_z}"/>
-      <geometry><box size="${body_l} ${body_w} ${body_h}"/></geometry>
-      <material name="dark"/>
-    </visual>
-    <collision>
-      <origin xyz="${body_x} 0 ${body_z}"/>
-      <geometry><box size="${body_l} ${body_w} ${body_h}"/></geometry>
-    </collision>
-    <!-- ponytail: 합친 부품(상판 0.2 · 적재함 0.05 · 폴 0.1kg) 질량은 본체 상자 하나에 더함 — 무게중심이 정확해야 하면 나눠 계산 -->
-    <xacro:box_inertia m="1.85" x="${body_l}" y="${body_w}" z="${body_h}"><origin xyz="${body_x} 0 ${body_z}"/></xacro:box_inertia>
-    <!-- 뒤쪽 캐스터 2개 (구, 충돌만) -->
-    <collision>
-      <origin xyz="${body_x - body_l / 2 + 0.020} 0.064 0.000"/>
-      <geometry><sphere radius="0.010"/></geometry>
-    </collision>
-    <collision>
-      <origin xyz="${body_x - body_l / 2 + 0.020} -0.064 0.000"/>
-      <geometry><sphere radius="0.010"/></geometry>
-    </collision>
-    <!-- 상판 (앞쪽 절반, 스탠드오프 위) — 윗면 z = deck_top -->
-    <xacro:part xyz="${deck_x} 0 ${deck_top - deck_t / 2}" material="white"><geometry><box size="${deck_l} ${body_w} ${deck_t}"/></geometry></xacro:part>
-    <collision>
-      <origin xyz="${deck_x} 0 ${deck_top - deck_t / 2}"/>
-      <geometry><box size="${deck_l} ${body_w} ${deck_t}"/></geometry>
-    </collision>
-    <xacro:macro name="standoff" params="x y">
-      <xacro:part xyz="${deck_x + x} ${y} ${deck_top - deck_t - deck_standoff / 2}" material="grey"><geometry><cylinder radius="0.004" length="${deck_standoff}"/></geometry></xacro:part>
-    </xacro:macro>
-    <xacro:standoff x="${deck_l / 2 - 0.01}" y="${body_w / 2 - 0.01}"/>
-    <xacro:standoff x="${deck_l / 2 - 0.01}" y="${-body_w / 2 + 0.01}"/>
-    <xacro:standoff x="${-deck_l / 2 + 0.01}" y="${body_w / 2 - 0.01}"/>
-    <xacro:standoff x="${-deck_l / 2 + 0.01}" y="${-body_w / 2 + 0.01}"/>
-    <!-- 적재함: 바닥판 + 가이드벽 4면 -->
-    <xacro:part xyz="-0.13 0 0.1375" material="grey"><geometry><box size="0.12 0.20 0.005"/></geometry></xacro:part>
-    <xacro:part xyz="-0.1875 0 0.16" material="grey"><geometry><box size="0.005 0.20 0.04"/></geometry></xacro:part>
-    <xacro:part xyz="-0.0725 0 0.16" material="grey"><geometry><box size="0.005 0.20 0.04"/></geometry></xacro:part>
-    <xacro:part xyz="-0.13 0.0975 0.16" material="grey"><geometry><box size="0.11 0.005 0.04"/></geometry></xacro:part>
-    <xacro:part xyz="-0.13 -0.0975 0.16" material="grey"><geometry><box size="0.11 0.005 0.04"/></geometry></xacro:part>
-    <collision>
-      <origin xyz="-0.13 0 0.1375"/>
-      <geometry><box size="0.12 0.20 0.005"/></geometry>
-    </collision>
-    <!-- 선가이드 폴 (뒤쪽 끝, 전원선이 위에서 내려옴) -->
-    <xacro:part xyz="${pole_x} 0 ${body_top + pole_h / 2}" material="grey"><geometry><cylinder radius="${pole_r}" length="${pole_h}"/></geometry></xacro:part>
-    <collision>
-      <origin xyz="${pole_x} 0 ${body_top + pole_h / 2}"/>
-      <geometry><cylinder radius="${pole_r}" length="${pole_h}"/></geometry>
-    </collision>
-  </link>
   <joint name="base_joint" type="fixed">
     <parent link="base_footprint"/>
     <child link="base_link"/>
-    <origin xyz="0 0 0.010"/>
-  </joint>
-  <xacro:macro name="wheel" params="side y">
-    <link name="wheel_${side}_link">
-      <visual>
-        <origin rpy="${-PI/2} 0 0"/>
-        <geometry><cylinder radius="${wheel_radius}" length="${wheel_width}"/></geometry>
-        <material name="grey"/>
-      </visual>
-      <collision>
-        <origin rpy="${-PI/2} 0 0"/>
-        <geometry><cylinder radius="${wheel_radius}" length="${wheel_width}"/></geometry>
-      </collision>
-      <xacro:cylinder_inertia m="0.03" r="${wheel_radius}" h="${wheel_width}"><origin rpy="${-PI/2} 0 0"/></xacro:cylinder_inertia>
-    </link>
-    <joint name="wheel_${side}_joint" type="continuous">
-      <parent link="base_link"/>
-      <child link="wheel_${side}_link"/>
-      <origin xyz="0 ${y} ${wheel_radius - 0.010}"/>
-      <axis xyz="0 1 0"/>
-    </joint>
-  </xacro:macro>
-  <xacro:wheel side="left" y="${wheel_separation / 2}"/>
-  <xacro:wheel side="right" y="${-wheel_separation / 2}"/>
-  <link name="imu_link"/>
-  <joint name="imu_joint" type="fixed">
-    <parent link="base_link"/>
-    <child link="imu_link"/>
-    <origin xyz="${body_x} 0 0.068"/>
-  </joint>
-  <!-- 카메라: <이름>_link (x 앞) + <이름>_color_optical_frame (z 앞 · x 오른쪽 · y 아래) — RealSense 드라이버 publish_tf는 끈다 -->
-  <xacro:macro name="camera" params="name parent *origin">
-    <link name="${name}_link">
-      <visual>
-        <geometry><box size="0.025 0.090 0.025"/></geometry>
-        <material name="blue"/>
-      </visual>
-      <collision><geometry><box size="0.025 0.090 0.025"/></geometry></collision>
-      <xacro:box_inertia m="0.07" x="0.025" y="0.090" z="0.025"><origin xyz="0 0 0"/></xacro:box_inertia>
-    </link>
-    <joint name="${name}_joint" type="fixed">
-      <parent link="${parent}"/>
-      <child link="${name}_link"/>
-      <xacro:insert_block name="origin"/>
-    </joint>
-    <link name="${name}_color_optical_frame"/>
-    <joint name="${name}_optical_joint" type="fixed">
-      <parent link="${name}_link"/>
-      <child link="${name}_color_optical_frame"/>
-      <origin rpy="${-PI/2} 0 ${-PI/2}"/>
-    </joint>
-  </xacro:macro>
-  <xacro:camera name="pole_cam" parent="base_link">
-    <origin xyz="${pole_x + 0.020} 0 ${body_top + pole_h}" rpy="0 0.6 0"/>   <!-- 폴 꼭대기 앞, 전방 하향 약 34° -->
-  </xacro:camera>
-  <!-- ================= 매니퓰레이터 (상판 위): OpenMANIPULATOR-X + 손목 roll 축 + 그리퍼 =================
-       관절 원점·축·한계·질량은 ROBOTIS open_manipulator (main) open_manipulator_x_arm.urdf.xacro 값 그대로,
-       joint4(손목 pitch)와 그리퍼 사이에 joint5(손목 roll, x축)를 끼웠다. 모양은 메시 대신 상자 (더미).
-          arm_base_link(베이스) ─joint1 yaw─ shoulder_link ─joint2 pitch─ upper_arm_link ─joint3 pitch─ forearm_link ─joint4 pitch─ wrist_link
-         ─joint5 roll(추가)─ gripper_link ─ gripper_left/right_joint(프리즘 → finger_left/right_link, 오른쪽은 mimic) · end_effector_link
-       gripper_cam(RealSense)은 gripper_link 위에 얹는다. -->
-  <xacro:macro name="box_link" params="name size xyz mass color:=orange">
-    <link name="${name}">
-      <visual>
-        <origin xyz="${xyz}"/>
-        <geometry><box size="${size}"/></geometry>
-        <material name="${color}"/>
-      </visual>
-      <collision>
-        <origin xyz="${xyz}"/>
-        <geometry><box size="${size}"/></geometry>
-      </collision>
-      <inertial>
-        <origin xyz="${xyz}"/>
-        <mass value="${mass}"/>
-        <inertia ixx="1e-4" ixy="0" ixz="0" iyy="1e-4" iyz="0" izz="1e-4"/>
-      </inertial>
-    </link>
-  </xacro:macro>
-  <!-- XM430-W350: 무부하 약 4.8rad/s (OM-X URDF velocity 4.8), stall 토크 약 4.1Nm -->
-  <xacro:macro name="arm_joint" params="name parent child xyz axis lower upper">
-    <joint name="${name}" type="revolute">
-      <parent link="${parent}"/>
-      <child link="${child}"/>
-      <origin xyz="${xyz}"/>
-      <axis xyz="${axis}"/>
-      <limit lower="${lower}" upper="${upper}" effort="4.1" velocity="4.8"/>
-    </joint>
-  </xacro:macro>
-  <xacro:property name="arm_mount_h" value="0.030"/>  <!-- 상판 위 joint1 높이 (베이스 서보) -->
-  <xacro:box_link name="arm_base_link" size="0.050 0.045 ${arm_mount_h}" xyz="0.012 0 ${-arm_mount_h / 2}" mass="0.079"/>
+    <origin rpy="0.000000 -0.000000 0.000000" xyz="0.000000 0.000000 0.010000"/>
+  </joint>
+  <link name="base_link">
+    <inertial>
+      <origin rpy="0 0 0" xyz="-0.085631 -0.000202 0.080552"/>
+      <mass value="2.400600"/>
+      <inertia ixx="2.8115e-02" ixy="-1.1729e-05" ixz="6.3963e-03" iyy="3.2571e-02" iyz="-7.6014e-06" izz="2.7719e-02"/>
+    </inertial>
+    <visual>
+      <origin rpy="0 0 0" xyz="0 0 0"/>
+      <geometry>
+        <mesh filename="$(arg mesh_uri)/base_link.stl" scale="0.001 0.001 0.001"/>
+      </geometry>
+    </visual>
+    <collision>
+      <origin rpy="0.000000 0.000000 0.000000" xyz="-0.081850 0.000000 0.045500"/>
+      <geometry>
+        <box size="0.301300 0.265600 0.091000"/>
+      </geometry>
+    </collision>
+    <collision>
+      <origin rpy="0.000000 0.000000 0.000000" xyz="0.032000 0.000000 0.108675"/>
+      <geometry>
+        <box size="0.073600 0.137600 0.035350"/>
+      </geometry>
+    </collision>
+    <collision>
+      <origin rpy="0.000000 0.000000 0.000000" xyz="-0.209400 0.000000 0.108675"/>
+      <geometry>
+        <box size="0.020000 0.020000 0.035350"/>
+      </geometry>
+    </collision>
+    <collision>
+      <origin rpy="0.000000 0.000000 0.000000" xyz="0.032000 0.000000 0.131250"/>
+      <geometry>
+        <box size="0.073600 0.137600 0.009800"/>
+      </geometry>
+    </collision>
+    <collision>
+      <origin rpy="0.000000 0.000000 0.000000" xyz="-0.209400 0.000000 0.291900"/>
+      <geometry>
+        <box size="0.020000 0.020000 0.331100"/>
+      </geometry>
+    </collision>
+    <collision>
+      <origin rpy="0 0 0" xyz="-0.177000 0.064000 -0.005237"/>
+      <geometry>
+        <sphere radius="0.004763"/>
+      </geometry>
+    </collision>
+    <collision>
+      <origin rpy="0 0 0" xyz="-0.177000 -0.064000 -0.005237"/>
+      <geometry>
+        <sphere radius="0.004763"/>
+      </geometry>
+    </collision>
+    <collision name="storage_collision_0">
+      <origin rpy="1.570796 0.000000 0.000000" xyz="-0.064000 0.000000 -0.000500"/>
+      <geometry>
+        <mesh filename="$(arg mesh_uri)/storage_collision/storage_0.stl" scale="0.001 0.001 0.001"/>
+      </geometry>
+    </collision>
+    <collision name="storage_collision_1">
+      <origin rpy="1.570796 0.000000 0.000000" xyz="-0.064000 0.000000 -0.000500"/>
+      <geometry>
+        <mesh filename="$(arg mesh_uri)/storage_collision/storage_1.stl" scale="0.001 0.001 0.001"/>
+      </geometry>
+    </collision>
+    <collision name="storage_collision_2">
+      <origin rpy="1.570796 0.000000 0.000000" xyz="-0.064000 0.000000 -0.000500"/>
+      <geometry>
+        <mesh filename="$(arg mesh_uri)/storage_collision/storage_2.stl" scale="0.001 0.001 0.001"/>
+      </geometry>
+    </collision>
+    <collision name="storage_collision_3">
+      <origin rpy="1.570796 0.000000 0.000000" xyz="-0.064000 0.000000 -0.000500"/>
+      <geometry>
+        <mesh filename="$(arg mesh_uri)/storage_collision/storage_3.stl" scale="0.001 0.001 0.001"/>
+      </geometry>
+    </collision>
+    <collision name="storage_collision_4">
+      <origin rpy="1.570796 0.000000 0.000000" xyz="-0.064000 0.000000 -0.000500"/>
+      <geometry>
+        <mesh filename="$(arg mesh_uri)/storage_collision/storage_4.stl" scale="0.001 0.001 0.001"/>
+      </geometry>
+    </collision>
+    <collision name="storage_collision_5">
+      <origin rpy="1.570796 0.000000 0.000000" xyz="-0.064000 0.000000 -0.000500"/>
+      <geometry>
+        <mesh filename="$(arg mesh_uri)/storage_collision/storage_5.stl" scale="0.001 0.001 0.001"/>
+      </geometry>
+    </collision>
+    <collision name="storage_collision_6">
+      <origin rpy="1.570796 0.000000 0.000000" xyz="-0.064000 0.000000 -0.000500"/>
+      <geometry>
+        <mesh filename="$(arg mesh_uri)/storage_collision/storage_6.stl" scale="0.001 0.001 0.001"/>
+      </geometry>
+    </collision>
+    <collision name="storage_collision_7">
+      <origin rpy="1.570796 0.000000 0.000000" xyz="-0.064000 0.000000 -0.000500"/>
+      <geometry>
+        <mesh filename="$(arg mesh_uri)/storage_collision/storage_7.stl" scale="0.001 0.001 0.001"/>
+      </geometry>
+    </collision>
+    <collision name="storage_collision_8">
+      <origin rpy="1.570796 0.000000 0.000000" xyz="-0.064000 0.000000 -0.000500"/>
+      <geometry>
+        <mesh filename="$(arg mesh_uri)/storage_collision/storage_8.stl" scale="0.001 0.001 0.001"/>
+      </geometry>
+    </collision>
+  </link>
+  <joint name="wheel_left_joint" type="continuous">
+    <parent link="base_link"/>
+    <child link="wheel_left_link"/>
+    <origin rpy="0.000000 -0.000000 0.000000" xyz="0.000000 0.143900 0.023000"/>
+    <axis xyz="0 1 0"/>
+    <limit effort="3.0" velocity="8.063"/>
+  </joint>
+  <link name="wheel_left_link">
+    <inertial>
+      <origin rpy="0 0 0" xyz="0.000000 -0.000704 0.000002"/>
+      <mass value="0.028500"/>
+      <inertia ixx="1.1098e-05" ixy="5.7318e-09" ixz="3.1818e-09" iyy="2.0549e-05" iyz="-4.8114e-11" izz="1.1095e-05"/>
+    </inertial>
+    <visual>
+      <origin rpy="0 0 0" xyz="0 0 0"/>
+      <geometry>
+        <mesh filename="$(arg mesh_uri)/wheel_left_link.stl" scale="0.001 0.001 0.001"/>
+      </geometry>
+    </visual>
+    <collision>
+      <origin rpy="1.570796 0 0" xyz="0 0 0"/>
+      <geometry>
+        <cylinder length="0.018200" radius="0.033000"/>
+      </geometry>
+    </collision>
+  </link>
+  <joint name="wheel_right_joint" type="continuous">
+    <parent link="base_link"/>
+    <child link="wheel_right_link"/>
+    <origin rpy="0.000000 -0.000000 0.000000" xyz="0.000000 -0.143900 0.023000"/>
+    <axis xyz="0 1 0"/>
+    <limit effort="3.0" velocity="8.063"/>
+  </joint>
+  <link name="wheel_right_link">
+    <inertial>
+      <origin rpy="0 0 0" xyz="0.000000 0.000704 -0.000002"/>
+      <mass value="0.028500"/>
+      <inertia ixx="1.1098e-05" ixy="-5.7318e-09" ixz="-3.1818e-09" iyy="2.0549e-05" iyz="-4.8114e-11" izz="1.1095e-05"/>
+    </inertial>
+    <visual>
+      <origin rpy="0 0 0" xyz="0 0 0"/>
+      <geometry>
+        <mesh filename="$(arg mesh_uri)/wheel_right_link.stl" scale="0.001 0.001 0.001"/>
+      </geometry>
+    </visual>
+    <collision>
+      <origin rpy="1.570796 0 0" xyz="0 0 0"/>
+      <geometry>
+        <cylinder length="0.018200" radius="0.033000"/>
+      </geometry>
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