Commit message: feat: v00 urdf fix

File: lv2_module6/urdf/beebot_slam/urdf.xacro (robot description, xacro)
@@ -1,200 +1,544 @@
-<?xml version="1.0"?>
+<?xml version="1.0" ?>
 <!--
-  beebot (SLAM 전용) — 지도 스캔할 때 쓰는 모델: 팔·그리퍼·gripper_cam을 떼고, 폴 위 카메라를 앞뒤 두 대로 (더미 치수)
-    beebot_normal/urdf.xacro 에서: 매니퓰레이터(arm_base_link ~ finger·end_effector · gripper_cam)와 ros2_control 팔 관절 6개 삭제,
-    폴 꼭대기 반대편(뒤)에 pole_rear_cam 추가 — pole_cam은 앞 아래, pole_rear_cam은 뒤 아래를 같은 각도(34°)로 본다.
-    남은 링크·관절 이름은 beebot_mesh · beebot_normal과 같다 (pole_rear_cam만 이 모델에 새로)
+  beebot — 실측 CAD(bee.urdf, SolidWorks 내보내기)에서 만든 모델. bee.urdf를 새로 받으면 이 파일을 다시 만든다:
+    · 메시 경로: meshes/x.stl → meshes/x.stl
+    · 이름 맞춤(제어·시뮬레이터가 쓰는 이름): camera_rear → front_pole_cam, camera_wrist → gripper_cam,
+      gripper_joint → gripper_left_joint, gripper_mimic_joint → gripper_right_joint, tcp → end_effector
+    · 추가: imu_link · <ros2_control> 블록(BeebotSystemHardware) · xacro 인자
   설계: documents/ros2-design/07-tf.md (TF 트리), 08-ctrl.md (ros2_control)
   좌표: base_footprint(바닥) → base_link(바퀴 축 아래 0.010m), x 앞 · y 왼쪽 · z 위
-    - 차체: Waffle Pi 본체 266×266mm, 바퀴 반경 0.033m · 간격 0.287m, 뒤쪽 캐스터 2개
-    - 상판(deck): 차체 위 앞쪽 절반만 덮는 판넬, 스탠드오프 0.05m 위
-    - 매니퓰레이터: 없음 (SLAM 전용 — 상판은 그대로)
-    - 선가이드 폴: 차체 위 뒤쪽 끝, 전원선이 위에서 내려온다. 폴 꼭대기 앞쪽에 pole_cam(전방 하향) · 뒤쪽에 pole_rear_cam(후방 하향)
+  구동 관절 6개: joint1~5 (팔) · gripper_left_joint (평행 그리퍼, 0=닫힘 · 0.0265=열림, 오른쪽은 mimic) + 바퀴 2개
   xacro 인자:
     mock_hardware (false)  true면 control/BeebotSystemHardware가 실기 대신 명령을 그대로 상태로 되돌려 줌 (테스트베드)
-    mock_effort   (0.0)    (팔이 없어 안 씀 — 다른 모델과 인자를 맞추려고 남김)
+    mock_effort   (0.0)    mock일 때 팔 관절 effort[A] (arm_safety_monitor 시험용)
     port          (/dev/opencr)  OpenCR 포트 (udev 고정 이름 — ros2_ws/99-opencr.rules)
-  TODO(권형중): 실측 치수·질량, pole_rear_cam 실제 장착 위치·각도
-  Isaac Sim용 USD는 이 파일을 xacro로 펼친 URDF를 Isaac Sim URDF Importer로 변환해 만든다:
-    xacro beebot.urdf.xacro > beebot.urdf
 -->
+<!-- generated by make_xacro.py -->
 <robot name="beebot" xmlns:xacro="http://www.ros.org/wiki/xacro">
   <xacro:arg name="mock_hardware" default="false"/>
   <xacro:arg name="mock_effort" default="0.0"/>
   <xacro:arg name="port" default="/dev/opencr"/>
-  <xacro:property name="PI" value="3.14159265"/>
-  <!-- 차체 -->
-  <xacro:property name="wheel_radius" value="0.033"/>
-  <xacro:property name="wheel_width" value="0.018"/>
-  <xacro:property name="wheel_separation" value="0.287"/>
-  <xacro:property name="body_l" value="0.266"/>
-  <xacro:property name="body_w" value="0.266"/>
-  <xacro:property name="body_h" value="0.110"/>
-  <xacro:property name="body_x" value="-0.064"/>   <!-- 바퀴 축 기준 본체 중심 (바퀴가 앞쪽) -->
-  <xacro:property name="body_z" value="0.080"/>
-  <xacro:property name="body_top" value="${body_z + body_h / 2}"/>
-  <!-- 상판: 본체 앞쪽 절반 -->
-  <xacro:property name="deck_standoff" value="0.050"/>
-  <xacro:property name="deck_t" value="0.005"/>
-  <xacro:property name="deck_l" value="${body_l / 2}"/>
-  <xacro:property name="deck_x" value="${body_x + body_l / 4}"/>
-  <xacro:property name="deck_top" value="${body_top + deck_standoff + deck_t}"/>
-  <!-- 선가이드 폴: 본체 뒤쪽 끝 -->
-  <xacro:property name="pole_h" value="0.450"/>
-  <xacro:property name="pole_r" value="0.010"/>
-  <xacro:property name="pole_x" value="${body_x - body_l / 2 + 0.020}"/>
-  <material name="dark"><color rgba="0.2 0.2 0.2 1"/></material>
-  <material name="grey"><color rgba="0.6 0.6 0.6 1"/></material>
-  <material name="white"><color rgba="0.95 0.95 0.95 1"/></material>
-  <material name="orange"><color rgba="0.95 0.5 0.1 1"/></material>
-  <material name="blue"><color rgba="0.2 0.4 0.8 1"/></material>
-  <!-- 관성: 균질 직육면체·원기둥·구 -->
-  <xacro:macro name="box_inertia" params="m x y z *origin">
-    <inertial>
-      <xacro:insert_block name="origin"/>
-      <mass value="${m}"/>
-      <inertia ixx="${m * (y*y + z*z) / 12}" ixy="0" ixz="0" iyy="${m * (x*x + z*z) / 12}" iyz="0" izz="${m * (x*x + y*y) / 12}"/>
-    </inertial>
-  </xacro:macro>
-  <xacro:macro name="cylinder_inertia" params="m r h *origin">
-    <inertial>
-      <xacro:insert_block name="origin"/>
-      <mass value="${m}"/>
-      <inertia ixx="${m * (3*r*r + h*h) / 12}" ixy="0" ixz="0" iyy="${m * (3*r*r + h*h) / 12}" iyz="0" izz="${m * r * r / 2}"/>
-    </inertial>
-  </xacro:macro>
-  <!-- ================= 베이스 =================
-       링크·관절 이름과 TF 트리는 beebot_mesh/urdf.xacro와 같다 (모델을 바꿔 끼워도 노드·설정이 그대로 돎).
-       beebot_mesh처럼 차체에 붙은 것(캐스터·상판·적재함·선가이드 폴)은 base_link 한 링크의 도형으로 합쳤다. -->
-  <!-- 적재함 (뒤쪽 절반, 퍽 운반): 바닥 윗면 z=0.140 (base_link 기준) · 가이드벽 4면 (높이 0.04, 두께 0.005)
-       시뮬레이터는 같은 치수로 퍽 받침·가둠 판정 (simulator/main.py TRAY) -->
-  <xacro:property name="tray_x0" value="-0.19"/>
-  <xacro:property name="tray_x1" value="-0.07"/>
-  <xacro:property name="tray_y" value="0.10"/>
-  <xacro:property name="tray_floor_z" value="0.140"/>
-  <xacro:property name="tray_wall_h" value="0.04"/>
-  <xacro:property name="tray_wall_t" value="0.005"/>
-  <xacro:macro name="part" params="xyz *geometry material">
-    <visual>
-      <origin xyz="${xyz}"/>
-      <xacro:insert_block name="geometry"/>
-      <material name="${material}"/>
-    </visual>
-  </xacro:macro>
+  <xacro:arg name="mesh_uri" default="package://ros_system/urdf/meshes"/>
   <link name="base_footprint"/>
-  <link name="base_link">
-    <!-- 본체 -->
-    <visual>
-      <origin xyz="${body_x} 0 ${body_z}"/>
-      <geometry><box size="${body_l} ${body_w} ${body_h}"/></geometry>
-      <material name="dark"/>
-    </visual>
-    <collision>
-      <origin xyz="${body_x} 0 ${body_z}"/>
-      <geometry><box size="${body_l} ${body_w} ${body_h}"/></geometry>
-    </collision>
-    <!-- ponytail: 합친 부품(상판 0.2 · 적재함 0.05 · 폴 0.1kg) 질량은 본체 상자 하나에 더함 — 무게중심이 정확해야 하면 나눠 계산 -->
-    <xacro:box_inertia m="1.85" x="${body_l}" y="${body_w}" z="${body_h}"><origin xyz="${body_x} 0 ${body_z}"/></xacro:box_inertia>
-    <!-- 뒤쪽 캐스터 2개 (구, 충돌만) -->
-    <collision>
-      <origin xyz="${body_x - body_l / 2 + 0.020} 0.064 0.000"/>
-      <geometry><sphere radius="0.010"/></geometry>
-    </collision>
-    <collision>
-      <origin xyz="${body_x - body_l / 2 + 0.020} -0.064 0.000"/>
-      <geometry><sphere radius="0.010"/></geometry>
-    </collision>
-    <!-- 상판 (앞쪽 절반, 스탠드오프 위) — 윗면 z = deck_top -->
-    <xacro:part xyz="${deck_x} 0 ${deck_top - deck_t / 2}" material="white"><geometry><box size="${deck_l} ${body_w} ${deck_t}"/></geometry></xacro:part>
-    <collision>
-      <origin xyz="${deck_x} 0 ${deck_top - deck_t / 2}"/>
-      <geometry><box size="${deck_l} ${body_w} ${deck_t}"/></geometry>
-    </collision>
-    <xacro:macro name="standoff" params="x y">
-      <xacro:part xyz="${deck_x + x} ${y} ${deck_top - deck_t - deck_standoff / 2}" material="grey"><geometry><cylinder radius="0.004" length="${deck_standoff}"/></geometry></xacro:part>
-    </xacro:macro>
-    <xacro:standoff x="${deck_l / 2 - 0.01}" y="${body_w / 2 - 0.01}"/>
-    <xacro:standoff x="${deck_l / 2 - 0.01}" y="${-body_w / 2 + 0.01}"/>
-    <xacro:standoff x="${-deck_l / 2 + 0.01}" y="${body_w / 2 - 0.01}"/>
-    <xacro:standoff x="${-deck_l / 2 + 0.01}" y="${-body_w / 2 + 0.01}"/>
-    <!-- 적재함: 바닥판 + 가이드벽 4면 -->
-    <xacro:part xyz="-0.13 0 0.1375" material="grey"><geometry><box size="0.12 0.20 0.005"/></geometry></xacro:part>
-    <xacro:part xyz="-0.1875 0 0.16" material="grey"><geometry><box size="0.005 0.20 0.04"/></geometry></xacro:part>
-    <xacro:part xyz="-0.0725 0 0.16" material="grey"><geometry><box size="0.005 0.20 0.04"/></geometry></xacro:part>
-    <xacro:part xyz="-0.13 0.0975 0.16" material="grey"><geometry><box size="0.11 0.005 0.04"/></geometry></xacro:part>
-    <xacro:part xyz="-0.13 -0.0975 0.16" material="grey"><geometry><box size="0.11 0.005 0.04"/></geometry></xacro:part>
-    <collision>
-      <origin xyz="-0.13 0 0.1375"/>
-      <geometry><box size="0.12 0.20 0.005"/></geometry>
-    </collision>
-    <!-- 선가이드 폴 (뒤쪽 끝, 전원선이 위에서 내려옴) -->
-    <xacro:part xyz="${pole_x} 0 ${body_top + pole_h / 2}" material="grey"><geometry><cylinder radius="${pole_r}" length="${pole_h}"/></geometry></xacro:part>
-    <collision>
-      <origin xyz="${pole_x} 0 ${body_top + pole_h / 2}"/>
-      <geometry><cylinder radius="${pole_r}" length="${pole_h}"/></geometry>
-    </collision>
-  </link>
   <joint name="base_joint" type="fixed">
     <parent link="base_footprint"/>
     <child link="base_link"/>
-    <origin xyz="0 0 0.010"/>
-  </joint>
-  <xacro:macro name="wheel" params="side y">
-    <link name="wheel_${side}_link">
-      <visual>
-        <origin rpy="${-PI/2} 0 0"/>
-        <geometry><cylinder radius="${wheel_radius}" length="${wheel_width}"/></geometry>
-        <material name="grey"/>
-      </visual>
-      <collision>
-        <origin rpy="${-PI/2} 0 0"/>
-        <geometry><cylinder radius="${wheel_radius}" length="${wheel_width}"/></geometry>
-      </collision>
-      <xacro:cylinder_inertia m="0.03" r="${wheel_radius}" h="${wheel_width}"><origin rpy="${-PI/2} 0 0"/></xacro:cylinder_inertia>
-    </link>
-    <joint name="wheel_${side}_joint" type="continuous">
-      <parent link="base_link"/>
-      <child link="wheel_${side}_link"/>
-      <origin xyz="0 ${y} ${wheel_radius - 0.010}"/>
-      <axis xyz="0 1 0"/>
-    </joint>
-  </xacro:macro>
-  <xacro:wheel side="left" y="${wheel_separation / 2}"/>
-  <xacro:wheel side="right" y="${-wheel_separation / 2}"/>
+    <origin rpy="0.000000 -0.000000 0.000000" xyz="0.000000 0.000000 0.010000"/>
+  </joint>
+  <link name="base_link">
+    <inertial>
+      <origin rpy="0 0 0" xyz="-0.085631 -0.000202 0.080552"/>
+      <mass value="2.400600"/>
+      <inertia ixx="2.8115e-02" ixy="-1.1729e-05" ixz="6.3963e-03" iyy="3.2571e-02" iyz="-7.6014e-06" izz="2.7719e-02"/>
+    </inertial>
+    <visual>
+      <origin rpy="0 0 0" xyz="0 0 0"/>
+      <geometry>
+        <mesh filename="$(arg mesh_uri)/base_link.stl" scale="0.001 0.001 0.001"/>
+      </geometry>
+    </visual>
+    <collision>
+      <origin rpy="0.000000 0.000000 0.000000" xyz="-0.081850 0.000000 0.045500"/>
+      <geometry>
+        <box size="0.301300 0.265600 0.091000"/>
+      </geometry>
+    </collision>
+    <collision>
+      <origin rpy="0.000000 0.000000 0.000000" xyz="0.032000 0.000000 0.108675"/>
+      <geometry>
+        <box size="0.073600 0.137600 0.035350"/>
+      </geometry>
+    </collision>
+    <collision>
+      <origin rpy="0.000000 0.000000 0.000000" xyz="-0.209400 0.000000 0.108675"/>
+      <geometry>
+        <box size="0.020000 0.020000 0.035350"/>
+      </geometry>
+    </collision>
+    <collision>
+      <origin rpy="0.000000 0.000000 0.000000" xyz="0.032000 0.000000 0.131250"/>
+      <geometry>
+        <box size="0.073600 0.137600 0.009800"/>
+      </geometry>
+    </collision>
+    <collision>
+      <origin rpy="0.000000 0.000000 0.000000" xyz="-0.209400 0.000000 0.291900"/>
+      <geometry>
+        <box size="0.020000 0.020000 0.331100"/>
+      </geometry>
+    </collision>
+    <collision>
+      <origin rpy="0 0 0" xyz="-0.177000 0.064000 -0.005237"/>
+      <geometry>
+        <sphere radius="0.004763"/>
+      </geometry>
+    </collision>
+    <collision>
+      <origin rpy="0 0 0" xyz="-0.177000 -0.064000 -0.005237"/>
+      <geometry>
+        <sphere radius="0.004763"/>
+      </geometry>
+    </collision>
+    <collision name="storage_collision_0">
+      <origin rpy="1.570796 0.000000 0.000000" xyz="-0.064000 0.000000 -0.000500"/>
+      <geometry>
+        <mesh filename="$(arg mesh_uri)/storage_collision/storage_0.stl" scale="0.001 0.001 0.001"/>
+      </geometry>
+    </collision>
+    <collision name="storage_collision_1">
+      <origin rpy="1.570796 0.000000 0.000000" xyz="-0.064000 0.000000 -0.000500"/>
+      <geometry>
+        <mesh filename="$(arg mesh_uri)/storage_collision/storage_1.stl" scale="0.001 0.001 0.001"/>
+      </geometry>
+    </collision>
+    <collision name="storage_collision_2">
+      <origin rpy="1.570796 0.000000 0.000000" xyz="-0.064000 0.000000 -0.000500"/>
+      <geometry>
+        <mesh filename="$(arg mesh_uri)/storage_collision/storage_2.stl" scale="0.001 0.001 0.001"/>
+      </geometry>
+    </collision>
+    <collision name="storage_collision_3">
+      <origin rpy="1.570796 0.000000 0.000000" xyz="-0.064000 0.000000 -0.000500"/>
+      <geometry>
+        <mesh filename="$(arg mesh_uri)/storage_collision/storage_3.stl" scale="0.001 0.001 0.001"/>
+      </geometry>
+    </collision>
+    <collision name="storage_collision_4">
+      <origin rpy="1.570796 0.000000 0.000000" xyz="-0.064000 0.000000 -0.000500"/>
+      <geometry>
+        <mesh filename="$(arg mesh_uri)/storage_collision/storage_4.stl" scale="0.001 0.001 0.001"/>
+      </geometry>
+    </collision>
+    <collision name="storage_collision_5">
+      <origin rpy="1.570796 0.000000 0.000000" xyz="-0.064000 0.000000 -0.000500"/>
+      <geometry>
+        <mesh filename="$(arg mesh_uri)/storage_collision/storage_5.stl" scale="0.001 0.001 0.001"/>
+      </geometry>
+    </collision>
+    <collision name="storage_collision_6">
+      <origin rpy="1.570796 0.000000 0.000000" xyz="-0.064000 0.000000 -0.000500"/>
+      <geometry>
+        <mesh filename="$(arg mesh_uri)/storage_collision/storage_6.stl" scale="0.001 0.001 0.001"/>
+      </geometry>
+    </collision>
+    <collision name="storage_collision_7">
+      <origin rpy="1.570796 0.000000 0.000000" xyz="-0.064000 0.000000 -0.000500"/>
+      <geometry>
+        <mesh filename="$(arg mesh_uri)/storage_collision/storage_7.stl" scale="0.001 0.001 0.001"/>
+      </geometry>
+    </collision>
+    <collision name="storage_collision_8">
+      <origin rpy="1.570796 0.000000 0.000000" xyz="-0.064000 0.000000 -0.000500"/>
+      <geometry>
+        <mesh filename="$(arg mesh_uri)/storage_collision/storage_8.stl" scale="0.001 0.001 0.001"/>
+      </geometry>
+    </collision>
+  </link>
+  <joint name="wheel_left_joint" type="continuous">
+    <parent link="base_link"/>
+    <child link="wheel_left_link"/>
+    <origin rpy="0.000000 -0.000000 0.000000" xyz="0.000000 0.143900 0.023000"/>
+    <axis xyz="0 1 0"/>
+    <limit effort="3.0" velocity="8.063"/>
+  </joint>
+  <link name="wheel_left_link">
+    <inertial>
+      <origin rpy="0 0 0" xyz="0.000000 -0.000704 0.000002"/>
+      <mass value="0.028500"/>
+      <inertia ixx="1.1098e-05" ixy="5.7318e-09" ixz="3.1818e-09" iyy="2.0549e-05" iyz="-4.8114e-11" izz="1.1095e-05"/>
+    </inertial>
+    <visual>
+      <origin rpy="0 0 0" xyz="0 0 0"/>
+      <geometry>
+        <mesh filename="$(arg mesh_uri)/wheel_left_link.stl" scale="0.001 0.001 0.001"/>
+      </geometry>
+    </visual>
+    <collision>
+      <origin rpy="1.570796 0 0" xyz="0 0 0"/>
+      <geometry>
+        <cylinder length="0.018200" radius="0.033000"/>
+      </geometry>
+    </collision>
+  </link>
+  <joint name="wheel_right_joint" type="continuous">
+    <parent link="base_link"/>
+    <child link="wheel_right_link"/>
+    <origin rpy="0.000000 -0.000000 0.000000" xyz="0.000000 -0.143900 0.023000"/>
+    <axis xyz="0 1 0"/>
+    <limit effort="3.0" velocity="8.063"/>
+  </joint>
+  <link name="wheel_right_link">
+    <inertial>
+      <origin rpy="0 0 0" xyz="0.000000 0.000704 -0.000002"/>
+      <mass value="0.028500"/>
+      <inertia ixx="1.1098e-05" ixy="-5.7318e-09" ixz="-3.1818e-09" iyy="2.0549e-05" iyz="-4.8114e-11" izz="1.1095e-05"/>
+    </inertial>
+    <visual>
+      <origin rpy="0 0 0" xyz="0 0 0"/>
+      <geometry>
+        <mesh filename="$(arg mesh_uri)/wheel_right_link.stl" scale="0.001 0.001 0.001"/>
+      </geometry>
+    </visual>
+    <collision>
+      <origin rpy="1.570796 0 0" xyz="0 0 0"/>
+      <geometry>
+        <cylinder length="0.018200" radius="0.033000"/>
+      </geometry>
+    </collision>
+  </link>
+  <joint name="front_pole_cam_joint" type="fixed">
+    <parent link="base_link"/>
+    <child link="front_pole_cam_link"/>
+    <origin rpy="0.000000 0.314159 0.000000" xyz="-0.137869 0.000185 0.434932"/>
+  </joint>
+  <link name="front_pole_cam_link">
+    <inertial>
+      <origin rpy="0 0 0" xyz="-0.013393 0.001408 -0.000023"/>
+      <mass value="0.072000"/>
+      <inertia ixx="4.6203e-05" ixy="4.1597e-07" ixz="2.0009e-08" iyy="6.9218e-06" iyz="3.6648e-09" izz="4.6614e-05"/>
+    </inertial>
+    <visual>
+      <origin rpy="0 0 0" xyz="0 0 0"/>
+      <geometry>
+        <mesh filename="$(arg mesh_uri)/camera_rear_link.stl" scale="0.001 0.001 0.001"/>
+      </geometry>
+    </visual>
+    <collision>
+      <origin rpy="0.000000 0.000000 0.000000" xyz="-0.012525 -0.000058 -0.000000"/>
+      <geometry>
+        <box size="0.025050 0.089714 0.025000"/>
+      </geometry>
+    </collision>
+  </link>
+  <joint name="arm_mount_joint" type="fixed">
+    <parent link="base_link"/>
+    <child link="arm_base_link"/>
+    <origin rpy="-0.000000 0.000000 0.000000" xyz="0.047985 -0.00023 0.130175"/>
+  </joint>
+  <link name="arm_base_link">
+    <inertial>
+      <origin rpy="0.0 0.0 0.0" xyz="-0.01169226743052282 -3.774353380840405e-15 0.023926534323405226"/>
+      <mass value="0.08108257974970318"/>
+      <inertia ixx="1.2862502962900217e-05" ixy="6.251056457349735e-19" ixz="-1.811662342359175e-07" iyy="2.2531969968508323e-05" iyz="1.5086560978736273e-17" izz="1.9821050957242446e-05"/>
+    </inertial>
+    <visual name="arm_base_link_visual">
+      <origin rpy="0.0 -0.0 0.0" xyz="0.0 0.0 0.0"/>
+      <geometry>
+        <mesh filename="$(arg mesh_uri)/arm_base_1.stl" scale="0.001 0.001 0.001"/>
+      </geometry>
+    </visual>
+    <collision name="arm_base_link_collision">
+      <origin rpy="0.0 -0.0 0.0" xyz="0.0 0.0 0.0"/>
+      <geometry>
+        <mesh filename="$(arg mesh_uri)/arm_base_1.stl" scale="0.001 0.001 0.001"/>
+      </geometry>
+    </collision>
+  </link>
+  <link name="shoulder_link">
+    <inertial>
+      <origin rpy="0.0 -0.0 0.0" xyz="1.3576596988624524e-13 0.0006685783443131954 0.028869490461060965"/>
+      <mass value="0.08583374201044289"/>
+      <inertia ixx="2.6324742259425243e-05" ixy="-7.312006911381859e-16" ixz="-9.128905585988183e-18" iyy="2.2861624315008813e-05" iyz="-8.980408739570743e-08" izz="1.4187591495603722e-05"/>
+    </inertial>
+    <visual name="shoulder_link_visual">
+      <origin rpy="-2.220438457117713e-16 -0.0 0.0" xyz="2.493290125897981e-18 -9.081593289611446e-18 -0.0409"/>
+      <geometry>
+        <mesh filename="$(arg mesh_uri)/shoulder_1.stl" scale="0.001 0.001 0.001"/>
+      </geometry>
+    </visual>
+    <collision name="shoulder_link_collision">
+      <origin rpy="-2.220438457117713e-16 -0.0 0.0" xyz="2.493290125897981e-18 -9.081593289611446e-18 -0.0409"/>
+      <geometry>
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