Commit message: fix: urdf v00 fix

File: lv2_module6/urdf/beebot_mesh/beebot.urdf (robot description, URDF)
Before this commit: robot beebot, 30 links, 29 joints
Links:
- removed link pole_cam_color_optical_frame
- removed link pole_cam_link
- added link front_pole_cam_color_optical_frame
- added link front_pole_cam_link, mass 0.072000; collision box size=0.025050 0.089714 0.025000; visual mesh filename=meshes/camera_rear_link.stl scale=0.001 0.001 0.001
- link arm_base_link: geometry collision mesh filename=meshes/arm_base_1.stl scale=0.001 0.001 0.001; visual mesh filename=meshes/arm_base_1.stl scale=0.001 0.001 0.001
- link base_link: geometry collision box size=0.020000 0.020000 0.035350; collision box size=0.020000 0.020000 0.331100
- link finger_left_link: geometry collision mesh filename=meshes/finger_R_1.stl scale=0.001 0.001 0.001; visual mesh filename=meshes/finger_R_1.stl scale=0.001 0.001 0.001
- link finger_right_link: geometry collision mesh filename=meshes/finger_L_1.stl scale=0.001 0.001 0.001; visual mesh filename=meshes/finger_L_1.stl scale=0.001 0.001 0.001
- link forearm_link: geometry collision mesh filename=meshes/link2_1.stl scale=0.001 0.001 0.001; visual mesh filename=meshes/link2_1.stl scale=0.001 0.001 0.001
- link gripper_cam_link: geometry collision box size=0.055050 0.089714 0.045413; visual mesh filename=meshes/camera_wrist_link.stl scale=0.001 0.001 0.001
- link gripper_link: geometry collision mesh filename=meshes/gripper_body_1.stl scale=0.001 0.001 0.001; visual mesh filename=meshes/gripper_body_1.stl scale=0.001 0.001 0.001
- link shoulder_link: geometry collision mesh filename=meshes/shoulder_1.stl scale=0.001 0.001 0.001; visual mesh filename=meshes/shoulder_1.stl scale=0.001 0.001 0.001
- link upper_arm_link: geometry collision mesh filename=meshes/link1_1.stl scale=0.001 0.001 0.001; visual mesh filename=meshes/link1_1.stl scale=0.001 0.001 0.001
- link wheel_left_link: geometry collision cylinder length=0.018200 radius=0.033000; visual mesh filename=meshes/wheel_left_link.stl scale=0.001 0.001 0.001
- link wheel_right_link: geometry collision cylinder length=0.018200 radius=0.033000; visual mesh filename=meshes/wheel_right_link.stl scale=0.001 0.001 0.001
- link wrist_link: geometry collision mesh filename=meshes/wrist_1.stl scale=0.001 0.001 0.001; visual mesh filename=meshes/wrist_1.stl scale=0.001 0.001 0.001
Joints:
- removed joint pole_cam_joint
- removed joint pole_cam_optical_joint
- added joint front_pole_cam_joint: type fixed, parent base_link, child front_pole_cam_link, origin xyz=-0.137869 0.000185 0.434932 rpy=0.000000 0.314159 0.000000
- added joint front_pole_cam_optical_joint: type fixed, parent front_pole_cam_link, child front_pole_cam_color_optical_frame, origin xyz=-0.004300 0.032500 0.000000 rpy=-1.570796 0.000000 -1.570796

File: lv2_module6/urdf/beebot_mesh/urdf.xacro (robot description, xacro)
@@ -3,5 +3,5 @@
   beebot — 실측 CAD(bee.urdf, SolidWorks 내보내기)에서 만든 모델. bee.urdf를 새로 받으면 이 파일을 다시 만든다:
     · 메시 경로: meshes/x.stl → meshes/x.stl
-    · 이름 맞춤(제어·시뮬레이터가 쓰는 이름): camera_rear → pole_cam, camera_wrist → gripper_cam,
+    · 이름 맞춤(제어·시뮬레이터가 쓰는 이름): camera_rear → front_pole_cam, camera_wrist → gripper_cam,
       gripper_joint → gripper_left_joint, gripper_mimic_joint → gripper_right_joint, tcp → end_effector
     · 추가: imu_link · <ros2_control> 블록(BeebotSystemHardware) · xacro 인자
@@ -15,5 +15,9 @@
 -->
 <!-- generated by make_xacro.py -->
-<robot name="beebot">
+<robot name="beebot" xmlns:xacro="http://www.ros.org/wiki/xacro">
+  <xacro:arg name="mock_hardware" default="false"/>
+  <xacro:arg name="mock_effort" default="0.0"/>
+  <xacro:arg name="port" default="/dev/opencr"/>
+  <xacro:arg name="mesh_uri" default="package://ros_system/urdf/meshes"/>
   <link name="base_footprint"/>
   <joint name="base_joint" type="fixed">
@@ -183,10 +187,10 @@
     </collision>
   </link>
-  <joint name="pole_cam_joint" type="fixed">
-    <parent link="base_link"/>
-    <child link="pole_cam_link"/>
-    <origin rpy="0.000000 0.314159 0.000000" xyz="-0.137869 0.000185 0.417108"/>
-  </joint>
-  <link name="pole_cam_link">
+  <joint name="front_pole_cam_joint" type="fixed">
+    <parent link="base_link"/>
+    <child link="front_pole_cam_link"/>
+    <origin rpy="0.000000 0.314159 0.000000" xyz="-0.137869 0.000185 0.434932"/>
+  </joint>
+  <link name="front_pole_cam_link">
     <inertial>
       <origin rpy="0 0 0" xyz="-0.013393 0.001408 -0.000023"/>
@@ -444,11 +448,11 @@
   </joint>
   <link name="end_effector_link"/>
-  <joint name="pole_cam_optical_joint" type="fixed">
-    <parent link="pole_cam_link"/>
-    <child link="pole_cam_color_optical_frame"/>
+  <joint name="front_pole_cam_optical_joint" type="fixed">
+    <parent link="front_pole_cam_link"/>
+    <child link="front_pole_cam_color_optical_frame"/>
     <!-- D435 RGB lens: +32.5 mm left of body center, 4.3 mm behind front glass (realsense-ros _d435.urdf.xacro) -->
     <origin rpy="-1.570796 0.000000 -1.570796" xyz="-0.004300 0.032500 0.000000"/>
   </joint>
-  <link name="pole_cam_color_optical_frame"/>
+  <link name="front_pole_cam_color_optical_frame"/>
   <joint name="gripper_cam_optical_joint" type="fixed">
     <parent link="gripper_cam_link"/>
@@ -607,59 +611,3 @@
     </sensor>
   </ros2_control>
-  <!-- Gazebo (gz-sim): RGBD 카메라 2대. 센서는 optical 프레임 링크에 identity로 — 렌즈가 보는 방향 = optical +Z.
-       방향이 뒤집혀 보이면 sensor 안 <pose>에 rpy를 얹어 맞춘다 (URDF optical joint와 같은 값부터). -->
-  <gazebo reference="pole_cam_color_optical_frame">
-    <sensor name="pole_rgbd" type="rgbd_camera">
-      <always_on>true</always_on>
-      <update_rate>30</update_rate>
-      <topic>pole_cam/rgbd</topic>
-      <camera>
-        <horizontal_fov>1.204</horizontal_fov>
-        <image><width>640</width><height>480</height><format>R8G8B8</format></image>
-        <clip><near>0.1</near><far>10.0</far></clip>
-      </camera>
-    </sensor>
-  </gazebo>
-  <gazebo reference="gripper_cam_color_optical_frame">
-    <sensor name="gripper_rgbd" type="rgbd_camera">
-      <always_on>true</always_on>
-      <update_rate>15</update_rate>
-      <topic>gripper_cam/rgbd</topic>
-      <camera>
-        <horizontal_fov>1.204</horizontal_fov>
-        <image><width>640</width><height>480</height><format>R8G8B8</format></image>
-        <clip><near>0.1</near><far>10.0</far></clip>
-      </camera>
-    </sensor>
-  </gazebo>
-  <!-- Gazebo 차체 구동: DiffDrive 플러그인 (teleop → /gz/cmd_vel → 바퀴, /gz/odometry → /gz/odom 보기용).
-       토픽을 /cmd_vel·/odom이 아니라 /gz/* 로 둔 이유: 돌고 있는 testbed(mock 하드웨어) 토픽과 안 섞이게.
-       팔·그리퍼는 JointPositionController가 0에 고정 (중력에 접히지 않게).
-       TODO(제어): 본番은 gz_ros2_control + diff_drive_controller로 testbed 체인에 합류 -->
-  <gazebo>
-    <plugin filename="libgz-sim-diff-drive-system.so" name="gz::sim::systems::DiffDrive">
-      <left_joint>wheel_left_joint</left_joint>
-      <right_joint>wheel_right_joint</right_joint>
-      <wheel_separation>0.287</wheel_separation>
-      <wheel_radius>0.033</wheel_radius>
-      <min_velocity>-0.5</min_velocity>
-      <max_velocity>0.5</max_velocity>
-      <topic>/model/beebot/cmd_vel</topic>
-      <odom_topic>/model/beebot/odometry</odom_topic>
-      <frame_id>odom</frame_id>
-      <child_frame_id>base_footprint</child_frame_id>
-      <publish_odom_tf>false</publish_odom_tf>
-    </plugin>
-    <plugin filename="libgz-sim-joint-position-controller-system.so" name="gz::sim::systems::JointPositionController">
-      <joint_name>joint1</joint_name>
-      <joint_name>joint2</joint_name>
-      <joint_name>joint3</joint_name>
-      <joint_name>joint4</joint_name>
-      <joint_name>joint5</joint_name>
-      <joint_name>gripper_left_joint</joint_name>
-      <joint_name>gripper_right_joint</joint_name>
-      <initial_position>0</initial_position>
-      <p_gain>10</p_gain>
-    </plugin>
-  </gazebo>
 </robot>

File: lv2_module6/urdf/default/urdf.xacro (robot description, xacro)
@@ -3,5 +3,5 @@
   beebot — 실측 CAD(bee.urdf, SolidWorks 내보내기)에서 만든 모델. bee.urdf를 새로 받으면 이 파일을 다시 만든다:
     · 메시 경로: meshes/x.stl → meshes/x.stl
-    · 이름 맞춤(제어·시뮬레이터가 쓰는 이름): camera_rear → pole_cam, camera_wrist → gripper_cam,
+    · 이름 맞춤(제어·시뮬레이터가 쓰는 이름): camera_rear → front_pole_cam, camera_wrist → gripper_cam,
       gripper_joint → gripper_left_joint, gripper_mimic_joint → gripper_right_joint, tcp → end_effector
     · 추가: imu_link · <ros2_control> 블록(BeebotSystemHardware) · xacro 인자
@@ -187,10 +187,10 @@
     </collision>
   </link>
-  <joint name="pole_cam_joint" type="fixed">
-    <parent link="base_link"/>
-    <child link="pole_cam_link"/>
-    <origin rpy="0.000000 0.314159 0.000000" xyz="-0.137869 0.000185 0.417108"/>
-  </joint>
-  <link name="pole_cam_link">
+  <joint name="front_pole_cam_joint" type="fixed">
+    <parent link="base_link"/>
+    <child link="front_pole_cam_link"/>
+    <origin rpy="0.000000 0.314159 0.000000" xyz="-0.137869 0.000185 0.434932"/>
+  </joint>
+  <link name="front_pole_cam_link">
     <inertial>
       <origin rpy="0 0 0" xyz="-0.013393 0.001408 -0.000023"/>
@@ -448,11 +448,11 @@
   </joint>
   <link name="end_effector_link"/>
-  <joint name="pole_cam_optical_joint" type="fixed">
-    <parent link="pole_cam_link"/>
-    <child link="pole_cam_color_optical_frame"/>
+  <joint name="front_pole_cam_optical_joint" type="fixed">
+    <parent link="front_pole_cam_link"/>
+    <child link="front_pole_cam_color_optical_frame"/>
     <!-- D435 RGB lens: +32.5 mm left of body center, 4.3 mm behind front glass (realsense-ros _d435.urdf.xacro) -->
     <origin rpy="-1.570796 0.000000 -1.570796" xyz="-0.004300 0.032500 0.000000"/>
   </joint>
-  <link name="pole_cam_color_optical_frame"/>
+  <link name="front_pole_cam_color_optical_frame"/>
   <joint name="gripper_cam_optical_joint" type="fixed">
     <parent link="gripper_cam_link"/>
@@ -611,3 +611,59 @@
     </sensor>
   </ros2_control>
+  <!-- Gazebo (gz-sim): RGBD 카메라 2대. 센서는 optical 프레임 링크에 identity로 — 렌즈가 보는 방향 = optical +Z.
+       방향이 뒤집혀 보이면 sensor 안 <pose>에 rpy를 얹어 맞춘다 (URDF optical joint와 같은 값부터). -->
+  <gazebo reference="front_pole_cam_color_optical_frame">
+    <sensor name="pole_rgbd" type="rgbd_camera">
+      <always_on>true</always_on>
+      <update_rate>30</update_rate>
+      <topic>pole_cam/rgbd</topic>
+      <camera>
+        <horizontal_fov>1.204</horizontal_fov>
+        <image><width>640</width><height>480</height><format>R8G8B8</format></image>
+        <clip><near>0.1</near><far>10.0</far></clip>
+      </camera>
+    </sensor>
+  </gazebo>
+  <gazebo reference="gripper_cam_color_optical_frame">
+    <sensor name="gripper_rgbd" type="rgbd_camera">
+      <always_on>true</always_on>
+      <update_rate>15</update_rate>
+      <topic>gripper_cam/rgbd</topic>
+      <camera>
+        <horizontal_fov>1.204</horizontal_fov>
+        <image><width>640</width><height>480</height><format>R8G8B8</format></image>
+        <clip><near>0.1</near><far>10.0</far></clip>
+      </camera>
+    </sensor>
+  </gazebo>
+  <!-- Gazebo 차체 구동: DiffDrive 플러그인 (teleop → /gz/cmd_vel → 바퀴, /gz/odometry → /gz/odom 보기용).
+       토픽을 /cmd_vel·/odom이 아니라 /gz/* 로 둔 이유: 돌고 있는 testbed(mock 하드웨어) 토픽과 안 섞이게.
+       팔·그리퍼는 JointPositionController가 0에 고정 (중력에 접히지 않게).
+       TODO(제어): 본番은 gz_ros2_control + diff_drive_controller로 testbed 체인에 합류 -->
+  <gazebo>
+    <plugin filename="libgz-sim-diff-drive-system.so" name="gz::sim::systems::DiffDrive">
+      <left_joint>wheel_left_joint</left_joint>
+      <right_joint>wheel_right_joint</right_joint>
+      <wheel_separation>0.287</wheel_separation>
+      <wheel_radius>0.033</wheel_radius>
+      <min_velocity>-0.5</min_velocity>
+      <max_velocity>0.5</max_velocity>
+      <topic>/model/beebot/cmd_vel</topic>
+      <odom_topic>/model/beebot/odometry</odom_topic>
+      <frame_id>odom</frame_id>
+      <child_frame_id>base_footprint</child_frame_id>
+      <publish_odom_tf>false</publish_odom_tf>
+    </plugin>
+    <plugin filename="libgz-sim-joint-position-controller-system.so" name="gz::sim::systems::JointPositionController">
+      <joint_name>joint1</joint_name>
+      <joint_name>joint2</joint_name>
+      <joint_name>joint3</joint_name>
+      <joint_name>joint4</joint_name>
+      <joint_name>joint5</joint_name>
+      <joint_name>gripper_left_joint</joint_name>
+      <joint_name>gripper_right_joint</joint_name>
+      <initial_position>0</initial_position>
+      <p_gain>10</p_gain>
+    </plugin>
+  </gazebo>
 </robot>

Commit message: feat: urdf fix, scene_sim.usda setup

File: lv2_module6/urdf/beebot_mesh/beebot.urdf (robot description, URDF)
Before this commit: robot beebot, 30 links, 29 joints
Joints:
- joint pole_front_cam_joint: origin xyz=-0.137869 0.000185 0.417108 rpy=0.000000 0.314159 0.000000 -> xyz=-0.137869 0.000185 0.434932 rpy=0.000000 0.314159 0.000000

File: lv2_module6/urdf/beebot_mesh/urdf.xacro (robot description, xacro)
@@ -204,5 +204,5 @@
     <parent link="base_link"/>
     <child link="pole_front_cam_link"/>
-    <origin rpy="0.000000 0.314159 0.000000" xyz="-0.137869 0.000185 0.417108"/>
+    <origin rpy="0.000000 0.314159 0.000000" xyz="-0.137869 0.000185 0.434932"/>
   </joint>
   <link name="pole_front_cam_link">

File: lv2_module6/urdf/default/urdf.xacro (robot description, xacro)
@@ -220,5 +220,5 @@
     <parent link="base_link"/>
     <child link="pole_front_cam_link"/>
-    <origin rpy="0.000000 0.314159 0.000000" xyz="-0.137869 0.000185 0.417108"/>
+    <origin rpy="0.000000 0.314159 0.000000" xyz="-0.137869 0.000185 0.434932"/>
   </joint>
   <link name="pole_front_cam_link">
