Commit message: feat: usd, urdf  edit - HDRI, texture, collision

File: lv2_module6/urdf/beebot_mesh/beebot.urdf (robot description, URDF)
Before this commit: robot beebot, 30 links, 29 joints
Links:
- link gripper_cam_link: geometry collision box size=0.025050 0.089714 0.025000; visual mesh filename=meshes/camera_wrist_link.stl scale=0.001 0.001 0.001
- link wheel_left_link: geometry collision cylinder length=0.015000 radius=0.033000; visual mesh filename=meshes/wheel_left_link.stl scale=0.001 0.001 0.001
- link wheel_right_link: geometry collision cylinder length=0.015000 radius=0.033000; visual mesh filename=meshes/wheel_right_link.stl scale=0.001 0.001 0.001

File: lv2_module6/urdf/beebot_mesh/urdf.xacro (robot description, xacro)
@@ -171,5 +171,5 @@
       <origin rpy="1.570796 0 0" xyz="0 0 0"/>
       <geometry>
-        <cylinder length="0.018200" radius="0.033000"/>
+        <cylinder length="0.015000" radius="0.033000"/>
       </geometry>
     </collision>
@@ -197,5 +197,5 @@
       <origin rpy="1.570796 0 0" xyz="0 0 0"/>
       <geometry>
-        <cylinder length="0.018200" radius="0.033000"/>
+        <cylinder length="0.015000" radius="0.033000"/>
       </geometry>
     </collision>
@@ -228,5 +228,5 @@
     <parent link="base_link"/>
     <child link="arm_base_link"/>
-    <origin rpy="-0.000000 0.000000 0.000000" xyz="0.051045 -0.000000 0.134795"/>
+    <origin rpy="-0.000000 0.000000 0.000000" xyz="0.047985 -0.00023 0.130175"/>
   </joint>
   <link name="arm_base_link">
@@ -435,11 +435,11 @@
     <parent link="gripper_link"/>
     <child link="gripper_cam_link"/>
-    <origin rpy="2.852763 -1.567096 -1.282111" xyz="0.000504 -0.050245 0.080871"/>
+    <origin rpy="0.003448 -1.260182 1.567371" xyz="0.000273 -0.040325 0.081681"/>
   </joint>
   <link name="gripper_cam_link">
     <inertial>
-      <origin rpy="0 0 0" xyz="-0.018065 0.001229 -0.001118"/>
+      <origin rpy="0 0 0" xyz="-0.017727 0.001229 -0.001059"/>
       <mass value="0.088370"/>
-      <inertia ixx="5.1972e-05" ixy="6.5780e-08" ixz="-2.7719e-06" iyy="1.8951e-05" iyz="-6.0902e-08" izz="6.0643e-05"/>
+      <inertia ixx="5.1824e-05" ixy="8.5769e-08" ixz="-2.1898e-06" iyy="1.7218e-05" iyz="-5.7372e-08" izz="5.9057e-05"/>
     </inertial>
     <visual>
@@ -450,7 +450,7 @@
     </visual>
     <collision>
-      <origin rpy="0.000000 0.000000 0.000000" xyz="-0.027566 -0.000058 -0.009755"/>
-      <geometry>
-        <box size="0.055131 0.089714 0.044510"/>
+      <origin rpy="0.000000 0.000000 0.000000" xyz="-0.012525 -0.000058 0.000000"/>
+      <geometry>
+        <box size="0.025050 0.089714 0.025000"/>
       </geometry>
     </collision>
@@ -472,5 +472,6 @@
     <parent link="gripper_cam_link"/>
     <child link="gripper_cam_color_optical_frame"/>
-    <origin rpy="-1.570796 0.000000 -1.570796" xyz="0.000000 0.000000 0.000000"/>
+    <!-- D435 RGB lens: +32.5 mm left of body center, 4.3 mm behind front glass (realsense-ros _d435.urdf.xacro) -->
+    <origin rpy="-1.570796 0.000000 -1.570796" xyz="-0.004300 0.032500 0.000000"/>
   </joint>
   <link name="gripper_cam_color_optical_frame"/>
@@ -481,4 +482,77 @@
     <origin rpy="0 0 0" xyz="-0.064 0 0.068"/>
   </joint>
+  <!-- basket slots: cell floor center, 3 rows (x, pole -> arm) x 4 cols (y, -y -> +y) -->
+  <joint name="basket_slot_0_joint" type="fixed">
+    <parent link="base_link"/>
+    <child link="basket_slot_0"/>
+    <origin rpy="0 0 0" xyz="-0.16984 -0.0975 0.09125"/>
+  </joint>
+  <link name="basket_slot_0"/>
+  <joint name="basket_slot_1_joint" type="fixed">
+    <parent link="base_link"/>
+    <child link="basket_slot_1"/>
+    <origin rpy="0 0 0" xyz="-0.16984 -0.0325 0.09125"/>
+  </joint>
+  <link name="basket_slot_1"/>
+  <joint name="basket_slot_2_joint" type="fixed">
+    <parent link="base_link"/>
+    <child link="basket_slot_2"/>
+    <origin rpy="0 0 0" xyz="-0.16984 0.0325 0.09125"/>
+  </joint>
+  <link name="basket_slot_2"/>
+  <joint name="basket_slot_3_joint" type="fixed">
+    <parent link="base_link"/>
+    <child link="basket_slot_3"/>
+    <origin rpy="0 0 0" xyz="-0.16984 0.0975 0.09125"/>
+  </joint>
+  <link name="basket_slot_3"/>
+  <joint name="basket_slot_4_joint" type="fixed">
+    <parent link="base_link"/>
+    <child link="basket_slot_4"/>
+    <origin rpy="0 0 0" xyz="-0.10484 -0.0975 0.09125"/>
+  </joint>
+  <link name="basket_slot_4"/>
+  <joint name="basket_slot_5_joint" type="fixed">
+    <parent link="base_link"/>
+    <child link="basket_slot_5"/>
+    <origin rpy="0 0 0" xyz="-0.10484 -0.0325 0.09125"/>
+  </joint>
+  <link name="basket_slot_5"/>
+  <joint name="basket_slot_6_joint" type="fixed">
+    <parent link="base_link"/>
+    <child link="basket_slot_6"/>
+    <origin rpy="0 0 0" xyz="-0.10484 0.0325 0.09125"/>
+  </joint>
+  <link name="basket_slot_6"/>
+  <joint name="basket_slot_7_joint" type="fixed">
+    <parent link="base_link"/>
+    <child link="basket_slot_7"/>
+    <origin rpy="0 0 0" xyz="-0.10484 0.0975 0.09125"/>
+  </joint>
+  <link name="basket_slot_7"/>
+  <joint name="basket_slot_8_joint" type="fixed">
+    <parent link="base_link"/>
+    <child link="basket_slot_8"/>
+    <origin rpy="0 0 0" xyz="-0.03984 -0.0975 0.09125"/>
+  </joint>
+  <link name="basket_slot_8"/>
+  <joint name="basket_slot_9_joint" type="fixed">
+    <parent link="base_link"/>
+    <child link="basket_slot_9"/>
+    <origin rpy="0 0 0" xyz="-0.03984 -0.0325 0.09125"/>
+  </joint>
+  <link name="basket_slot_9"/>
+  <joint name="basket_slot_10_joint" type="fixed">
+    <parent link="base_link"/>
+    <child link="basket_slot_10"/>
+    <origin rpy="0 0 0" xyz="-0.03984 0.0325 0.09125"/>
+  </joint>
+  <link name="basket_slot_10"/>
+  <joint name="basket_slot_11_joint" type="fixed">
+    <parent link="base_link"/>
+    <child link="basket_slot_11"/>
+    <origin rpy="0 0 0" xyz="-0.03984 0.0975 0.09125"/>
+  </joint>
+  <link name="basket_slot_11"/>
   <!-- ================= ros2_control ================= -->
   <ros2_control name="BeebotSystem" type="system">

File: lv2_module6/urdf/default/urdf.xacro (robot description, xacro)
@@ -16,8 +16,4 @@
 <!-- generated by make_xacro.py -->
 <robot name="beebot" xmlns:xacro="http://www.ros.org/wiki/xacro">
-  <!-- 링크 색상 (STL에 색이 없어 Gazebo·RViz가 하얗게 나옴) -->
-  <material name="beebot_body"><color rgba="0.25 0.27 0.30 1.0"/></material>
-  <material name="beebot_dark"><color rgba="0.10 0.10 0.12 1.0"/></material>
-  <material name="beebot_arm"><color rgba="0.90 0.45 0.10 1.0"/></material>
   <xacro:arg name="mock_hardware" default="false"/>
   <xacro:arg name="mock_effort" default="0.0"/>
@@ -41,5 +37,4 @@
         <mesh filename="$(arg mesh_uri)/base_link.stl" scale="0.001 0.001 0.001"/>
       </geometry>
-      <material name="beebot_body"/>
     </visual>
     <collision>
@@ -104,5 +99,4 @@
         <mesh filename="$(arg mesh_uri)/storage_collision/storage_0.stl" scale="0.001 0.001 0.001"/>
       </geometry>
-      <material name="beebot_body"/>
     </collision>
     <collision name="storage_collision_1">
@@ -111,5 +105,4 @@
         <mesh filename="$(arg mesh_uri)/storage_collision/storage_1.stl" scale="0.001 0.001 0.001"/>
       </geometry>
-      <material name="beebot_body"/>
     </collision>
     <collision name="storage_collision_2">
@@ -118,5 +111,4 @@
         <mesh filename="$(arg mesh_uri)/storage_collision/storage_2.stl" scale="0.001 0.001 0.001"/>
       </geometry>
-      <material name="beebot_body"/>
     </collision>
     <collision name="storage_collision_3">
@@ -125,5 +117,4 @@
         <mesh filename="$(arg mesh_uri)/storage_collision/storage_3.stl" scale="0.001 0.001 0.001"/>
       </geometry>
-      <material name="beebot_body"/>
     </collision>
     <collision name="storage_collision_4">
@@ -132,5 +123,4 @@
         <mesh filename="$(arg mesh_uri)/storage_collision/storage_4.stl" scale="0.001 0.001 0.001"/>
       </geometry>
-      <material name="beebot_body"/>
     </collision>
     <collision name="storage_collision_5">
@@ -139,5 +129,4 @@
         <mesh filename="$(arg mesh_uri)/storage_collision/storage_5.stl" scale="0.001 0.001 0.001"/>
       </geometry>
-      <material name="beebot_body"/>
     </collision>
     <collision name="storage_collision_6">
@@ -146,5 +135,4 @@
         <mesh filename="$(arg mesh_uri)/storage_collision/storage_6.stl" scale="0.001 0.001 0.001"/>
       </geometry>
-      <material name="beebot_body"/>
     </collision>
     <collision name="storage_collision_7">
@@ -153,5 +141,4 @@
         <mesh filename="$(arg mesh_uri)/storage_collision/storage_7.stl" scale="0.001 0.001 0.001"/>
       </geometry>
-      <material name="beebot_body"/>
     </collision>
     <collision name="storage_collision_8">
@@ -160,5 +147,4 @@
         <mesh filename="$(arg mesh_uri)/storage_collision/storage_8.stl" scale="0.001 0.001 0.001"/>
       </geometry>
-      <material name="beebot_body"/>
     </collision>
   </link>
@@ -181,10 +167,9 @@
         <mesh filename="$(arg mesh_uri)/wheel_left_link.stl" scale="0.001 0.001 0.001"/>
       </geometry>
-      <material name="beebot_dark"/>
     </visual>
     <collision>
       <origin rpy="1.570796 0 0" xyz="0 0 0"/>
       <geometry>
-        <cylinder length="0.018200" radius="0.033000"/>
+        <cylinder length="0.015000" radius="0.033000"/>
       </geometry>
     </collision>
@@ -208,10 +193,9 @@
         <mesh filename="$(arg mesh_uri)/wheel_right_link.stl" scale="0.001 0.001 0.001"/>
       </geometry>
-      <material name="beebot_dark"/>
     </visual>
     <collision>
       <origin rpy="1.570796 0 0" xyz="0 0 0"/>
       <geometry>
-        <cylinder length="0.018200" radius="0.033000"/>
+        <cylinder length="0.015000" radius="0.033000"/>
       </geometry>
     </collision>
@@ -233,5 +217,4 @@
         <mesh filename="$(arg mesh_uri)/camera_rear_link.stl" scale="0.001 0.001 0.001"/>
       </geometry>
-      <material name="beebot_dark"/>
     </visual>
     <collision>
@@ -245,5 +228,5 @@
     <parent link="base_link"/>
     <child link="arm_base_link"/>
-    <origin rpy="-0.000000 0.000000 0.000000" xyz="0.051045 -0.000000 0.134795"/>
+    <origin rpy="-0.000000 0.000000 0.000000" xyz="0.047985 -0.00023 0.130175"/>
   </joint>
   <link name="arm_base_link">
@@ -258,5 +241,4 @@
         <mesh filename="$(arg mesh_uri)/arm_base_1.stl" scale="0.001 0.001 0.001"/>
       </geometry>
-      <material name="beebot_arm"/>
     </visual>
     <collision name="arm_base_link_collision">
@@ -265,5 +247,4 @@
         <mesh filename="$(arg mesh_uri)/arm_base_1.stl" scale="0.001 0.001 0.001"/>
       </geometry>
-      <material name="beebot_arm"/>
     </collision>
   </link>
@@ -279,5 +260,4 @@
         <mesh filename="$(arg mesh_uri)/shoulder_1.stl" scale="0.001 0.001 0.001"/>
       </geometry>
-      <material name="beebot_arm"/>
     </visual>
     <collision name="shoulder_link_collision">
@@ -286,5 +266,4 @@
         <mesh filename="$(arg mesh_uri)/shoulder_1.stl" scale="0.001 0.001 0.001"/>
       </geometry>
-      <material name="beebot_arm"/>
     </collision>
   </link>
@@ -300,5 +279,4 @@
         <mesh filename="$(arg mesh_uri)/link1_1.stl" scale="0.001 0.001 0.001"/>
       </geometry>
-      <material name="beebot_arm"/>
     </visual>
     <collision name="upper_arm_link_collision">
@@ -307,5 +285,4 @@
         <mesh filename="$(arg mesh_uri)/link1_1.stl" scale="0.001 0.001 0.001"/>
       </geometry>
-      <material name="beebot_arm"/>
     </collision>
   </link>
@@ -321,5 +298,4 @@
         <mesh filename="$(arg mesh_uri)/link2_1.stl" scale="0.001 0.001 0.001"/>
       </geometry>
-      <material name="beebot_arm"/>
     </visual>
     <collision name="forearm_link_collision">
@@ -328,5 +304,4 @@
         <mesh filename="$(arg mesh_uri)/link2_1.stl" scale="0.001 0.001 0.001"/>
       </geometry>
-      <material name="beebot_arm"/>
     </collision>
   </link>
@@ -342,5 +317,4 @@
         <mesh filename="$(arg mesh_uri)/wrist_1.stl" scale="0.001 0.001 0.001"/>
       </geometry>
-      <material name="beebot_arm"/>
     </visual>
     <collision name="wrist_link_collision">
@@ -349,5 +323,4 @@
         <mesh filename="$(arg mesh_uri)/wrist_1.stl" scale="0.001 0.001 0.001"/>
       </geometry>
-      <material name="beebot_arm"/>
     </collision>
   </link>
@@ -363,5 +336,4 @@
         <mesh filename="$(arg mesh_uri)/gripper_body_1.stl" scale="0.001 0.001 0.001"/>
       </geometry>
-      <material name="beebot_dark"/>
     </visual>
     <collision name="gripper_link_collision">
@@ -370,5 +342,4 @@
         <mesh filename="$(arg mesh_uri)/gripper_body_1.stl" scale="0.001 0.001 0.001"/>
       </geometry>
-      <material name="beebot_dark"/>
     </collision>
   </link>
@@ -384,5 +355,4 @@
         <mesh filename="$(arg mesh_uri)/finger_R_1.stl" scale="0.001 0.001 0.001"/>
       </geometry>
-      <material name="beebot_dark"/>
     </visual>
     <collision name="finger_left_link_collision">
@@ -391,5 +361,4 @@
         <mesh filename="$(arg mesh_uri)/finger_R_1.stl" scale="0.001 0.001 0.001"/>
       </geometry>
-      <material name="beebot_dark"/>
     </collision>
   </link>
@@ -405,5 +374,4 @@
         <mesh filename="$(arg mesh_uri)/finger_L_1.stl" scale="0.001 0.001 0.001"/>
       </geometry>
-      <material name="beebot_dark"/>
     </visual>
     <collision name="finger_right_link_collision">
@@ -412,5 +380,4 @@
         <mesh filename="$(arg mesh_uri)/finger_L_1.stl" scale="0.001 0.001 0.001"/>
       </geometry>
-      <material name="beebot_dark"/>
     </collision>
   </link>
@@ -468,11 +435,11 @@
     <parent link="gripper_link"/>
     <child link="gripper_cam_link"/>
-    <origin rpy="2.852763 -1.567096 -1.282111" xyz="0.000504 -0.050245 0.080871"/>
+    <origin rpy="0.003448 -1.260182 1.567371" xyz="0.000273 -0.040325 0.081681"/>
   </joint>
   <link name="gripper_cam_link">
     <inertial>
-      <origin rpy="0 0 0" xyz="-0.018065 0.001229 -0.001118"/>
+      <origin rpy="0 0 0" xyz="-0.017727 0.001229 -0.001059"/>
       <mass value="0.088370"/>
-      <inertia ixx="5.1972e-05" ixy="6.5780e-08" ixz="-2.7719e-06" iyy="1.8951e-05" iyz="-6.0902e-08" izz="6.0643e-05"/>
+      <inertia ixx="5.1824e-05" ixy="8.5769e-08" ixz="-2.1898e-06" iyy="1.7218e-05" iyz="-5.7372e-08" izz="5.9057e-05"/>
     </inertial>
     <visual>
@@ -481,10 +448,9 @@
         <mesh filename="$(arg mesh_uri)/camera_wrist_link.stl" scale="0.001 0.001 0.001"/>
       </geometry>
-      <material name="beebot_dark"/>
-    </visual>
-    <collision>
-      <origin rpy="0.000000 0.000000 0.000000" xyz="-0.027566 -0.000058 -0.009755"/>
-      <geometry>
-        <box size="0.055131 0.089714 0.044510"/>
+    </visual>
+    <collision>
+      <origin rpy="0.000000 0.000000 0.000000" xyz="-0.012525 -0.000058 0.000000"/>
+      <geometry>
+        <box size="0.025050 0.089714 0.025000"/>
       </geometry>
     </collision>
@@ -506,5 +472,6 @@
     <parent link="gripper_cam_link"/>
     <child link="gripper_cam_color_optical_frame"/>
-    <origin rpy="-1.570796 0.000000 -1.570796" xyz="0.000000 0.000000 0.000000"/>
+    <!-- D435 RGB lens: +32.5 mm left of body center, 4.3 mm behind front glass (realsense-ros _d435.urdf.xacro) -->
+    <origin rpy="-1.570796 0.000000 -1.570796" xyz="-0.004300 0.032500 0.000000"/>
   </joint>
   <link name="gripper_cam_color_optical_frame"/>
@@ -515,4 +482,77 @@
     <origin rpy="0 0 0" xyz="-0.064 0 0.068"/>
   </joint>
+  <!-- basket slots: cell floor center, 3 rows (x, pole -> arm) x 4 cols (y, -y -> +y) -->
+  <joint name="basket_slot_0_joint" type="fixed">
+    <parent link="base_link"/>
+    <child link="basket_slot_0"/>
+    <origin rpy="0 0 0" xyz="-0.16984 -0.0975 0.09125"/>
+  </joint>
+  <link name="basket_slot_0"/>
+  <joint name="basket_slot_1_joint" type="fixed">
+    <parent link="base_link"/>
+    <child link="basket_slot_1"/>
+    <origin rpy="0 0 0" xyz="-0.16984 -0.0325 0.09125"/>
+  </joint>
+  <link name="basket_slot_1"/>
+  <joint name="basket_slot_2_joint" type="fixed">
+    <parent link="base_link"/>
+    <child link="basket_slot_2"/>
+    <origin rpy="0 0 0" xyz="-0.16984 0.0325 0.09125"/>
+  </joint>
+  <link name="basket_slot_2"/>
+  <joint name="basket_slot_3_joint" type="fixed">
+    <parent link="base_link"/>
+    <child link="basket_slot_3"/>
+    <origin rpy="0 0 0" xyz="-0.16984 0.0975 0.09125"/>
+  </joint>
+  <link name="basket_slot_3"/>
+  <joint name="basket_slot_4_joint" type="fixed">
+    <parent link="base_link"/>
+    <child link="basket_slot_4"/>
+    <origin rpy="0 0 0" xyz="-0.10484 -0.0975 0.09125"/>
+  </joint>
+  <link name="basket_slot_4"/>
+  <joint name="basket_slot_5_joint" type="fixed">
+    <parent link="base_link"/>
+    <child link="basket_slot_5"/>
+    <origin rpy="0 0 0" xyz="-0.10484 -0.0325 0.09125"/>
+  </joint>
+  <link name="basket_slot_5"/>
+  <joint name="basket_slot_6_joint" type="fixed">
+    <parent link="base_link"/>
+    <child link="basket_slot_6"/>
+    <origin rpy="0 0 0" xyz="-0.10484 0.0325 0.09125"/>
+  </joint>
+  <link name="basket_slot_6"/>
+  <joint name="basket_slot_7_joint" type="fixed">
+    <parent link="base_link"/>
+    <child link="basket_slot_7"/>
+    <origin rpy="0 0 0" xyz="-0.10484 0.0975 0.09125"/>
+  </joint>
+  <link name="basket_slot_7"/>
+  <joint name="basket_slot_8_joint" type="fixed">
+    <parent link="base_link"/>
+    <child link="basket_slot_8"/>
+    <origin rpy="0 0 0" xyz="-0.03984 -0.0975 0.09125"/>
+  </joint>
+  <link name="basket_slot_8"/>
+  <joint name="basket_slot_9_joint" type="fixed">
+    <parent link="base_link"/>
+    <child link="basket_slot_9"/>
+    <origin rpy="0 0 0" xyz="-0.03984 -0.0325 0.09125"/>
+  </joint>
+  <link name="basket_slot_9"/>
+  <joint name="basket_slot_10_joint" type="fixed">
+    <parent link="base_link"/>
+    <child link="basket_slot_10"/>
+    <origin rpy="0 0 0" xyz="-0.03984 0.0325 0.09125"/>
+  </joint>
+  <link name="basket_slot_10"/>
+  <joint name="basket_slot_11_joint" type="fixed">
+    <parent link="base_link"/>
+    <child link="basket_slot_11"/>
+    <origin rpy="0 0 0" xyz="-0.03984 0.0975 0.09125"/>
+  </joint>
+  <link name="basket_slot_11"/>
   <!-- ================= ros2_control ================= -->
   <ros2_control name="BeebotSystem" type="system">
