Commit message: feat: isaac to ros nvblox setup

File: lv2_module6/urdf/beebot_mesh/beebot.urdf (robot description, URDF)
Before this commit: robot beebot, 30 links, 29 joints
Links:
- link base_link: geometry collision box size=0.020000 0.020000 0.035350; collision box size=0.020000 0.020000 0.331100
- link gripper_cam_link: geometry collision box size=0.025050 0.089714 0.025000; visual mesh filename=meshes/camera_wrist_link.stl scale=0.001 0.001 0.001
- link wheel_left_link: geometry collision cylinder length=0.015000 radius=0.033000; visual mesh filename=meshes/wheel_left_link.stl scale=0.001 0.001 0.001
- link wheel_right_link: geometry collision cylinder length=0.015000 radius=0.033000; visual mesh filename=meshes/wheel_right_link.stl scale=0.001 0.001 0.001
Joints:
- joint end_effector_joint: origin xyz=-0.000000 0.000000 0.109055 rpy=-0.000000 0.000000 1.570796 -> xyz=0.109055 -2.3367178972231404e-11 0.0 rpy=-1.5707963264201519 1.5707959999869179 -1.5707963266344216
- joint gripper_cam_joint: origin xyz=0.000273 -0.040325 0.081681 rpy=0.003448 -1.260182 1.567371 -> xyz=0.08168099999994151 -0.0002730000175021933 0.04032500000000001 rpy=-0.00014947924188481 0.3106124436433518 -0.0010995446528302402
- joint gripper_left_joint: axis -0.000000 0.000000 -1.000000 -> 0 1 0; origin xyz=-0.038613870011387864 0.0 0.053149999991726635 rpy=-1.4210854715201966e-14 1.5707963265658087 0 -> xyz=0.05315000000000042 0.03861386999999943 0.0 rpy=0.0 0.0 0.0
- joint gripper_right_joint: axis 0.000000 0.000000 -1.000000 -> 0 -1 0; origin xyz=0.03861386998861214 0.0 0.0531500000082734 rpy=3.141592653589779 1.5707963265658087 0 -> xyz=0.053149999999999614 -0.03861387000000057 0.0 rpy=0.0 0.0 0.0
- joint imu_joint: origin xyz=-0.064 0 0.068 rpy=0 0 0 -> xyz=0.0178 0 0.0585 rpy=0 0 0
- joint joint1: axis 0.0 2.220438457117713e-16 1.0 -> 0 0 1; origin xyz=0.0 0.0 0.0409 rpy=2.220438457117713e-16 -0.0 0.0 -> xyz=0.0 0.0 0.0409 rpy=0.0 0.0 0.0
- joint joint2: axis 2.1442092918336785e-10 -3.854694341498492e-13 1.0 -> 0 1 0; origin xyz=-2.53596257304049e-18 -0.018749999999999992 0.041600000000000005 rpy=1.5707963267945113 -8.260510339448073e-23 3.141592653375372 -> xyz=0.0 0.0 0.041599999999999984 rpy=0.0 0.0 0.0
- joint joint3: axis 2.1428325780447923e-10 1.4210854715201836e-14 1.0 -> 0 1 0; origin xyz=-0.024 0.128 5.195441854510818e-12 rpy=3.9968028886505105e-13 1.3767137888862427e-13 -8.564479437823846e-23 -> xyz=0.024 0.0 0.12800000000000003 rpy=0.0 0.0 0.0
- joint joint4: axis 2.14258832897939e-10 -1.0658141036401452e-14 1.0 -> 0 1 0; origin xyz=-0.12400000000000003 0.0 2.657112530002337e-11 rpy=-2.486899575160329e-14 2.442490654022833e-14 5.328402005082324e-24 -> xyz=0.12400000000000001 0.0 0.0 rpy=0.0 0.0 0.0
- joint joint5: axis -2.1425895896776037e-10 0.0 1.0 -> 1 0 0; origin xyz=-0.06289999999598264 -2.1316282072803005e-16 0.018750000013476882 rpy=-3.141592653589793 1.570796326794886 0 -> xyz=0.06290000000000001 0.0 0.0 rpy=0.0 0.0 0.0
- joint pole_front_cam_joint: origin xyz=-0.137869 0.000185 0.417108 rpy=0.000000 0.314159 0.000000 -> xyz=-0.137869 0.000185 0.434932 rpy=0.000000 0.314159 0.000000
