Commit message: feat: isaac to ros nvblox setup

File: lv2_module6/urdf/default/urdf.xacro (robot description, xacro)
@@ -16,8 +16,4 @@
 <!-- generated by make_xacro.py -->
 <robot name="beebot" xmlns:xacro="http://www.ros.org/wiki/xacro">
-  <!-- 링크 색상 (STL에 색이 없어 Gazebo·RViz가 하얗게 나옴) -->
-  <material name="beebot_body"><color rgba="0.25 0.27 0.30 1.0"/></material>
-  <material name="beebot_dark"><color rgba="0.10 0.10 0.12 1.0"/></material>
-  <material name="beebot_arm"><color rgba="0.90 0.45 0.10 1.0"/></material>
   <xacro:arg name="mock_hardware" default="false"/>
   <xacro:arg name="mock_effort" default="0.0"/>
@@ -32,5 +28,5 @@
   <link name="base_link">
     <inertial>
-      <origin rpy="0 0 0" xyz="-0.085426 -0.000171 0.080461"/>
+      <origin rpy="0 0 0" xyz="-0.050770 -0.000171 0.080461"/>  <!-- x: real balance pose 2026-10-28 (was -0.085426 from build.py) -->
       <mass value="2.400600"/>
       <inertia ixx="2.8130e-02" ixy="-2.1613e-05" ixz="6.4439e-03" iyy="3.2644e-02" iyz="-1.4858e-06" izz="2.7766e-02"/>
@@ -41,5 +37,4 @@
         <mesh filename="$(arg mesh_uri)/base_link.stl" scale="0.001 0.001 0.001"/>
       </geometry>
-      <material name="beebot_body"/>
     </visual>
     <collision>
@@ -85,18 +80,4 @@
       </geometry>
     </collision>
-    <!-- front caster (v01) -->
-    <collision>
-      <origin rpy="0 0 0" xyz="0.049600 0.064000 -0.005237"/>
-      <geometry>
-        <sphere radius="0.004763"/>
-      </geometry>
-    </collision>
-    <!-- front caster (v01) -->
-    <collision>
-      <origin rpy="0 0 0" xyz="0.049600 -0.064000 -0.005237"/>
-      <geometry>
-        <sphere radius="0.004763"/>
-      </geometry>
-    </collision>
     <collision name="storage_collision_0">
       <origin rpy="1.570796 0.000000 0.000000" xyz="-0.064000 0.000000 -0.000500"/>
@@ -104,5 +85,4 @@
         <mesh filename="$(arg mesh_uri)/storage_collision/storage_0.stl" scale="0.001 0.001 0.001"/>
       </geometry>
-      <material name="beebot_body"/>
     </collision>
     <collision name="storage_collision_1">
@@ -111,5 +91,4 @@
         <mesh filename="$(arg mesh_uri)/storage_collision/storage_1.stl" scale="0.001 0.001 0.001"/>
       </geometry>
-      <material name="beebot_body"/>
     </collision>
     <collision name="storage_collision_2">
@@ -118,5 +97,4 @@
         <mesh filename="$(arg mesh_uri)/storage_collision/storage_2.stl" scale="0.001 0.001 0.001"/>
       </geometry>
-      <material name="beebot_body"/>
     </collision>
     <collision name="storage_collision_3">
@@ -125,5 +103,4 @@
         <mesh filename="$(arg mesh_uri)/storage_collision/storage_3.stl" scale="0.001 0.001 0.001"/>
       </geometry>
-      <material name="beebot_body"/>
     </collision>
     <collision name="storage_collision_4">
@@ -132,5 +109,4 @@
         <mesh filename="$(arg mesh_uri)/storage_collision/storage_4.stl" scale="0.001 0.001 0.001"/>
       </geometry>
-      <material name="beebot_body"/>
     </collision>
     <collision name="storage_collision_5">
@@ -139,5 +115,4 @@
         <mesh filename="$(arg mesh_uri)/storage_collision/storage_5.stl" scale="0.001 0.001 0.001"/>
       </geometry>
-      <material name="beebot_body"/>
     </collision>
     <collision name="storage_collision_6">
@@ -146,5 +121,4 @@
         <mesh filename="$(arg mesh_uri)/storage_collision/storage_6.stl" scale="0.001 0.001 0.001"/>
       </geometry>
-      <material name="beebot_body"/>
     </collision>
     <collision name="storage_collision_7">
@@ -153,5 +127,4 @@
         <mesh filename="$(arg mesh_uri)/storage_collision/storage_7.stl" scale="0.001 0.001 0.001"/>
       </geometry>
-      <material name="beebot_body"/>
     </collision>
     <collision name="storage_collision_8">
@@ -160,5 +133,4 @@
         <mesh filename="$(arg mesh_uri)/storage_collision/storage_8.stl" scale="0.001 0.001 0.001"/>
       </geometry>
-      <material name="beebot_body"/>
     </collision>
   </link>
@@ -181,10 +153,9 @@
         <mesh filename="$(arg mesh_uri)/wheel_left_link.stl" scale="0.001 0.001 0.001"/>
       </geometry>
-      <material name="beebot_dark"/>
     </visual>
     <collision>
       <origin rpy="1.570796 0 0" xyz="0 0 0"/>
       <geometry>
-        <cylinder length="0.018200" radius="0.033000"/>
+        <cylinder length="0.015000" radius="0.033000"/>
       </geometry>
     </collision>
@@ -208,10 +179,9 @@
         <mesh filename="$(arg mesh_uri)/wheel_right_link.stl" scale="0.001 0.001 0.001"/>
       </geometry>
-      <material name="beebot_dark"/>
     </visual>
     <collision>
       <origin rpy="1.570796 0 0" xyz="0 0 0"/>
       <geometry>
-        <cylinder length="0.018200" radius="0.033000"/>
+        <cylinder length="0.015000" radius="0.033000"/>
       </geometry>
     </collision>
@@ -220,5 +190,5 @@
     <parent link="base_link"/>
     <child link="pole_front_cam_link"/>
-    <origin rpy="0.000000 0.314159 0.000000" xyz="-0.137869 0.000185 0.417108"/>
+    <origin rpy="0.000000 0.314159 0.000000" xyz="-0.137869 0.000185 0.434932"/>
   </joint>
   <link name="pole_front_cam_link">
@@ -233,5 +203,4 @@
         <mesh filename="$(arg mesh_uri)/camera_rear_link.stl" scale="0.001 0.001 0.001"/>
       </geometry>
-      <material name="beebot_dark"/>
     </visual>
     <collision>
@@ -245,5 +214,5 @@
     <parent link="base_link"/>
     <child link="arm_base_link"/>
-    <origin rpy="-0.000000 0.000000 0.000000" xyz="0.051045 -0.000000 0.134795"/>
+    <origin rpy="-0.000000 0.000000 0.000000" xyz="0.047985 -0.00023 0.130175"/>
   </joint>
   <link name="arm_base_link">
@@ -258,5 +227,4 @@
         <mesh filename="$(arg mesh_uri)/arm_base_1.stl" scale="0.001 0.001 0.001"/>
       </geometry>
-      <material name="beebot_arm"/>
     </visual>
     <collision name="arm_base_link_collision">
@@ -265,5 +233,4 @@
         <mesh filename="$(arg mesh_uri)/arm_base_1.stl" scale="0.001 0.001 0.001"/>
       </geometry>
-      <material name="beebot_arm"/>
     </collision>
   </link>
@@ -279,5 +246,4 @@
         <mesh filename="$(arg mesh_uri)/shoulder_1.stl" scale="0.001 0.001 0.001"/>
       </geometry>
-      <material name="beebot_arm"/>
     </visual>
     <collision name="shoulder_link_collision">
@@ -286,5 +252,4 @@
         <mesh filename="$(arg mesh_uri)/shoulder_1.stl" scale="0.001 0.001 0.001"/>
       </geometry>
-      <material name="beebot_arm"/>
     </collision>
   </link>
@@ -300,5 +265,4 @@
         <mesh filename="$(arg mesh_uri)/link1_1.stl" scale="0.001 0.001 0.001"/>
       </geometry>
-      <material name="beebot_arm"/>
     </visual>
     <collision name="upper_arm_link_collision">
@@ -307,5 +271,4 @@
         <mesh filename="$(arg mesh_uri)/link1_1.stl" scale="0.001 0.001 0.001"/>
       </geometry>
-      <material name="beebot_arm"/>
     </collision>
   </link>
@@ -321,5 +284,4 @@
         <mesh filename="$(arg mesh_uri)/link2_1.stl" scale="0.001 0.001 0.001"/>
       </geometry>
-      <material name="beebot_arm"/>
     </visual>
     <collision name="forearm_link_collision">
@@ -328,5 +290,4 @@
         <mesh filename="$(arg mesh_uri)/link2_1.stl" scale="0.001 0.001 0.001"/>
       </geometry>
-      <material name="beebot_arm"/>
     </collision>
   </link>
@@ -342,5 +303,4 @@
         <mesh filename="$(arg mesh_uri)/wrist_1.stl" scale="0.001 0.001 0.001"/>
       </geometry>
-      <material name="beebot_arm"/>
     </visual>
     <collision name="wrist_link_collision">
@@ -349,5 +309,4 @@
         <mesh filename="$(arg mesh_uri)/wrist_1.stl" scale="0.001 0.001 0.001"/>
       </geometry>
-      <material name="beebot_arm"/>
     </collision>
   </link>
@@ -363,5 +322,4 @@
         <mesh filename="$(arg mesh_uri)/gripper_body_1.stl" scale="0.001 0.001 0.001"/>
       </geometry>
-      <material name="beebot_dark"/>
     </visual>
     <collision name="gripper_link_collision">
@@ -370,5 +328,4 @@
         <mesh filename="$(arg mesh_uri)/gripper_body_1.stl" scale="0.001 0.001 0.001"/>
       </geometry>
-      <material name="beebot_dark"/>
     </collision>
   </link>
@@ -384,5 +341,4 @@
         <mesh filename="$(arg mesh_uri)/finger_R_1.stl" scale="0.001 0.001 0.001"/>
       </geometry>
-      <material name="beebot_dark"/>
     </visual>
     <collision name="finger_left_link_collision">
@@ -391,5 +347,4 @@
         <mesh filename="$(arg mesh_uri)/finger_R_1.stl" scale="0.001 0.001 0.001"/>
       </geometry>
-      <material name="beebot_dark"/>
     </collision>
   </link>
@@ -405,5 +360,4 @@
         <mesh filename="$(arg mesh_uri)/finger_L_1.stl" scale="0.001 0.001 0.001"/>
       </geometry>
-      <material name="beebot_dark"/>
     </visual>
     <collision name="finger_right_link_collision">
@@ -412,5 +366,4 @@
         <mesh filename="$(arg mesh_uri)/finger_L_1.stl" scale="0.001 0.001 0.001"/>
       </geometry>
-      <material name="beebot_dark"/>
     </collision>
   </link>
@@ -468,11 +421,11 @@
     <parent link="gripper_link"/>
     <child link="gripper_cam_link"/>
-    <origin rpy="2.852763 -1.567096 -1.282111" xyz="0.000504 -0.050245 0.080871"/>
+    <origin rpy="0.003448 -1.260182 1.567371" xyz="0.000273 -0.040325 0.081681"/>
   </joint>
   <link name="gripper_cam_link">
     <inertial>
-      <origin rpy="0 0 0" xyz="-0.018065 0.001229 -0.001118"/>
+      <origin rpy="0 0 0" xyz="-0.017727 0.001229 -0.001059"/>
       <mass value="0.088370"/>
-      <inertia ixx="5.1972e-05" ixy="6.5780e-08" ixz="-2.7719e-06" iyy="1.8951e-05" iyz="-6.0902e-08" izz="6.0643e-05"/>
+      <inertia ixx="5.1824e-05" ixy="8.5769e-08" ixz="-2.1898e-06" iyy="1.7218e-05" iyz="-5.7372e-08" izz="5.9057e-05"/>
     </inertial>
     <visual>
@@ -481,10 +434,9 @@
         <mesh filename="$(arg mesh_uri)/camera_wrist_link.stl" scale="0.001 0.001 0.001"/>
       </geometry>
-      <material name="beebot_dark"/>
-    </visual>
-    <collision>
-      <origin rpy="0.000000 0.000000 0.000000" xyz="-0.027566 -0.000058 -0.009755"/>
-      <geometry>
-        <box size="0.055131 0.089714 0.044510"/>
+    </visual>
+    <collision>
+      <origin rpy="0.000000 0.000000 0.000000" xyz="-0.012525 -0.000058 0.000000"/>
+      <geometry>
+        <box size="0.025050 0.089714 0.025000"/>
       </geometry>
     </collision>
@@ -514,5 +466,6 @@
     <parent link="gripper_cam_link"/>
     <child link="gripper_cam_color_optical_frame"/>
-    <origin rpy="-1.570796 0.000000 -1.570796" xyz="0.000000 0.000000 0.000000"/>
+    <!-- D435 RGB lens: +32.5 mm left of body center, 4.3 mm behind front glass (realsense-ros _d435.urdf.xacro) -->
+    <origin rpy="-1.570796 0.000000 -1.570796" xyz="-0.004300 0.032500 0.000000"/>
   </joint>
   <link name="gripper_cam_color_optical_frame"/>
@@ -527,6 +480,79 @@
     <parent link="base_link"/>
     <child link="imu_link"/>
-    <origin rpy="0 0 0" xyz="-0.064 0 0.068"/>
-  </joint>
+    <origin rpy="0 0 0" xyz="0.0178 0 0.0585"/>  <!-- x: waffle front edge 0.0688 - 0.051 (measured); z: OpenCR board top in base_link mesh -->
+  </joint>
+  <!-- basket slots: cell floor center, 3 rows (x, pole -> arm) x 4 cols (y, -y -> +y) -->
+  <joint name="basket_slot_0_joint" type="fixed">
+    <parent link="base_link"/>
+    <child link="basket_slot_0"/>
+    <origin rpy="0 0 0" xyz="-0.16984 -0.0975 0.09125"/>
+  </joint>
+  <link name="basket_slot_0"/>
+  <joint name="basket_slot_1_joint" type="fixed">
+    <parent link="base_link"/>
+    <child link="basket_slot_1"/>
+    <origin rpy="0 0 0" xyz="-0.16984 -0.0325 0.09125"/>
+  </joint>
+  <link name="basket_slot_1"/>
+  <joint name="basket_slot_2_joint" type="fixed">
+    <parent link="base_link"/>
+    <child link="basket_slot_2"/>
+    <origin rpy="0 0 0" xyz="-0.16984 0.0325 0.09125"/>
+  </joint>
+  <link name="basket_slot_2"/>
+  <joint name="basket_slot_3_joint" type="fixed">
+    <parent link="base_link"/>
+    <child link="basket_slot_3"/>
+    <origin rpy="0 0 0" xyz="-0.16984 0.0975 0.09125"/>
+  </joint>
+  <link name="basket_slot_3"/>
+  <joint name="basket_slot_4_joint" type="fixed">
+    <parent link="base_link"/>
+    <child link="basket_slot_4"/>
+    <origin rpy="0 0 0" xyz="-0.10484 -0.0975 0.09125"/>
+  </joint>
+  <link name="basket_slot_4"/>
+  <joint name="basket_slot_5_joint" type="fixed">
+    <parent link="base_link"/>
+    <child link="basket_slot_5"/>
+    <origin rpy="0 0 0" xyz="-0.10484 -0.0325 0.09125"/>
+  </joint>
+  <link name="basket_slot_5"/>
+  <joint name="basket_slot_6_joint" type="fixed">
+    <parent link="base_link"/>
+    <child link="basket_slot_6"/>
+    <origin rpy="0 0 0" xyz="-0.10484 0.0325 0.09125"/>
+  </joint>
+  <link name="basket_slot_6"/>
+  <joint name="basket_slot_7_joint" type="fixed">
+    <parent link="base_link"/>
+    <child link="basket_slot_7"/>
+    <origin rpy="0 0 0" xyz="-0.10484 0.0975 0.09125"/>
+  </joint>
+  <link name="basket_slot_7"/>
+  <joint name="basket_slot_8_joint" type="fixed">
+    <parent link="base_link"/>
+    <child link="basket_slot_8"/>
+    <origin rpy="0 0 0" xyz="-0.03984 -0.0975 0.09125"/>
+  </joint>
+  <link name="basket_slot_8"/>
+  <joint name="basket_slot_9_joint" type="fixed">
+    <parent link="base_link"/>
+    <child link="basket_slot_9"/>
+    <origin rpy="0 0 0" xyz="-0.03984 -0.0325 0.09125"/>
+  </joint>
+  <link name="basket_slot_9"/>
+  <joint name="basket_slot_10_joint" type="fixed">
+    <parent link="base_link"/>
+    <child link="basket_slot_10"/>
+    <origin rpy="0 0 0" xyz="-0.03984 0.0325 0.09125"/>
+  </joint>
+  <link name="basket_slot_10"/>
+  <joint name="basket_slot_11_joint" type="fixed">
+    <parent link="base_link"/>
+    <child link="basket_slot_11"/>
+    <origin rpy="0 0 0" xyz="-0.03984 0.0975 0.09125"/>
+  </joint>
+  <link name="basket_slot_11"/>
   <!-- ================= ros2_control ================= -->
   <ros2_control name="BeebotSystem" type="system">
