Commit message: chore: sync latest beebot from isaac-pick
Co-Authored-By: Claude Opus 5.5 <noreply@anthropic.com>

File: lv2_module6/urdf/default/urdf.xacro (robot description, xacro)
@@ -16,8 +16,4 @@
 <!-- generated by make_xacro.py -->
 <robot name="beebot" xmlns:xacro="http://www.ros.org/wiki/xacro">
-  <!-- 링크 색상 (STL에 색이 없어 Gazebo·RViz가 하얗게 나옴) -->
-  <material name="beebot_body"><color rgba="0.25 0.27 0.30 1.0"/></material>
-  <material name="beebot_dark"><color rgba="0.10 0.10 0.12 1.0"/></material>
-  <material name="beebot_arm"><color rgba="0.90 0.45 0.10 1.0"/></material>
   <xacro:arg name="mock_hardware" default="false"/>
   <xacro:arg name="mock_effort" default="0.0"/>
@@ -32,5 +28,5 @@
   <link name="base_link">
     <inertial>
-      <origin rpy="0 0 0" xyz="-0.085426 -0.000171 0.080461"/>
+      <origin rpy="0 0 0" xyz="-0.050770 -0.000171 0.080461"/>  <!-- x: real balance pose 2026-10-28 (was -0.085426 from build.py) -->
       <mass value="2.400600"/>
       <inertia ixx="2.8130e-02" ixy="-2.1613e-05" ixz="6.4439e-03" iyy="3.2644e-02" iyz="-1.4858e-06" izz="2.7766e-02"/>
@@ -41,5 +37,77 @@
         <mesh filename="$(arg mesh_uri)/base_link.stl" scale="0.001 0.001 0.001"/>
       </geometry>
-      <material name="beebot_body"/>
+    </visual>
+    <!-- storage_support x 12: outer 44.5, hole 34, 35 mm high, top 8 mm chamfered to 42 -->
+    <visual name="storage_support_0">
+      <origin rpy="0 0 0" xyz="-0.169840 -0.097500 0.091000"/>
+      <geometry>
+        <mesh filename="$(arg mesh_uri)/storage_support.stl" scale="0.001 0.001 0.001"/>
+      </geometry>
+    </visual>
+    <visual name="storage_support_1">
+      <origin rpy="0 0 0" xyz="-0.169840 -0.032500 0.091000"/>
+      <geometry>
+        <mesh filename="$(arg mesh_uri)/storage_support.stl" scale="0.001 0.001 0.001"/>
+      </geometry>
+    </visual>
+    <visual name="storage_support_2">
+      <origin rpy="0 0 0" xyz="-0.169840 0.032500 0.091000"/>
+      <geometry>
+        <mesh filename="$(arg mesh_uri)/storage_support.stl" scale="0.001 0.001 0.001"/>
+      </geometry>
+    </visual>
+    <visual name="storage_support_3">
+      <origin rpy="0 0 0" xyz="-0.169840 0.097500 0.091000"/>
+      <geometry>
+        <mesh filename="$(arg mesh_uri)/storage_support.stl" scale="0.001 0.001 0.001"/>
+      </geometry>
+    </visual>
+    <visual name="storage_support_4">
+      <origin rpy="0 0 0" xyz="-0.104840 -0.097500 0.091000"/>
+      <geometry>
+        <mesh filename="$(arg mesh_uri)/storage_support.stl" scale="0.001 0.001 0.001"/>
+      </geometry>
+    </visual>
+    <visual name="storage_support_5">
+      <origin rpy="0 0 0" xyz="-0.104840 -0.032500 0.091000"/>
+      <geometry>
+        <mesh filename="$(arg mesh_uri)/storage_support.stl" scale="0.001 0.001 0.001"/>
+      </geometry>
+    </visual>
+    <visual name="storage_support_6">
+      <origin rpy="0 0 0" xyz="-0.104840 0.032500 0.091000"/>
+      <geometry>
+        <mesh filename="$(arg mesh_uri)/storage_support.stl" scale="0.001 0.001 0.001"/>
+      </geometry>
+    </visual>
+    <visual name="storage_support_7">
+      <origin rpy="0 0 0" xyz="-0.104840 0.097500 0.091000"/>
+      <geometry>
+        <mesh filename="$(arg mesh_uri)/storage_support.stl" scale="0.001 0.001 0.001"/>
+      </geometry>
+    </visual>
+    <visual name="storage_support_8">
+      <origin rpy="0 0 0" xyz="-0.039840 -0.097500 0.091000"/>
+      <geometry>
+        <mesh filename="$(arg mesh_uri)/storage_support.stl" scale="0.001 0.001 0.001"/>
+      </geometry>
+    </visual>
+    <visual name="storage_support_9">
+      <origin rpy="0 0 0" xyz="-0.039840 -0.032500 0.091000"/>
+      <geometry>
+        <mesh filename="$(arg mesh_uri)/storage_support.stl" scale="0.001 0.001 0.001"/>
+      </geometry>
+    </visual>
+    <visual name="storage_support_10">
+      <origin rpy="0 0 0" xyz="-0.039840 0.032500 0.091000"/>
+      <geometry>
+        <mesh filename="$(arg mesh_uri)/storage_support.stl" scale="0.001 0.001 0.001"/>
+      </geometry>
+    </visual>
+    <visual name="storage_support_11">
+      <origin rpy="0 0 0" xyz="-0.039840 0.097500 0.091000"/>
+      <geometry>
+        <mesh filename="$(arg mesh_uri)/storage_support.stl" scale="0.001 0.001 0.001"/>
+      </geometry>
     </visual>
     <collision>
@@ -85,18 +153,4 @@
       </geometry>
     </collision>
-    <!-- front caster (v01) -->
-    <collision>
-      <origin rpy="0 0 0" xyz="0.049600 0.064000 -0.005237"/>
-      <geometry>
-        <sphere radius="0.004763"/>
-      </geometry>
-    </collision>
-    <!-- front caster (v01) -->
-    <collision>
-      <origin rpy="0 0 0" xyz="0.049600 -0.064000 -0.005237"/>
-      <geometry>
-        <sphere radius="0.004763"/>
-      </geometry>
-    </collision>
     <collision name="storage_collision_0">
       <origin rpy="1.570796 0.000000 0.000000" xyz="-0.064000 0.000000 -0.000500"/>
@@ -104,5 +158,4 @@
         <mesh filename="$(arg mesh_uri)/storage_collision/storage_0.stl" scale="0.001 0.001 0.001"/>
       </geometry>
-      <material name="beebot_body"/>
     </collision>
     <collision name="storage_collision_1">
@@ -111,5 +164,4 @@
         <mesh filename="$(arg mesh_uri)/storage_collision/storage_1.stl" scale="0.001 0.001 0.001"/>
       </geometry>
-      <material name="beebot_body"/>
     </collision>
     <collision name="storage_collision_2">
@@ -118,5 +170,4 @@
         <mesh filename="$(arg mesh_uri)/storage_collision/storage_2.stl" scale="0.001 0.001 0.001"/>
       </geometry>
-      <material name="beebot_body"/>
     </collision>
     <collision name="storage_collision_3">
@@ -125,5 +176,4 @@
         <mesh filename="$(arg mesh_uri)/storage_collision/storage_3.stl" scale="0.001 0.001 0.001"/>
       </geometry>
-      <material name="beebot_body"/>
     </collision>
     <collision name="storage_collision_4">
@@ -132,5 +182,4 @@
         <mesh filename="$(arg mesh_uri)/storage_collision/storage_4.stl" scale="0.001 0.001 0.001"/>
       </geometry>
-      <material name="beebot_body"/>
     </collision>
     <collision name="storage_collision_5">
@@ -139,5 +188,4 @@
         <mesh filename="$(arg mesh_uri)/storage_collision/storage_5.stl" scale="0.001 0.001 0.001"/>
       </geometry>
-      <material name="beebot_body"/>
     </collision>
     <collision name="storage_collision_6">
@@ -146,5 +194,4 @@
         <mesh filename="$(arg mesh_uri)/storage_collision/storage_6.stl" scale="0.001 0.001 0.001"/>
       </geometry>
-      <material name="beebot_body"/>
     </collision>
     <collision name="storage_collision_7">
@@ -153,5 +200,4 @@
         <mesh filename="$(arg mesh_uri)/storage_collision/storage_7.stl" scale="0.001 0.001 0.001"/>
       </geometry>
-      <material name="beebot_body"/>
     </collision>
     <collision name="storage_collision_8">
@@ -160,5 +206,292 @@
         <mesh filename="$(arg mesh_uri)/storage_collision/storage_8.stl" scale="0.001 0.001 0.001"/>
       </geometry>
-      <material name="beebot_body"/>
+    </collision>
+    <collision name="storage_support_0_0">
+      <origin rpy="0 0 0" xyz="-0.169840 -0.097500 0.091000"/>
+      <geometry>
+        <mesh filename="$(arg mesh_uri)/storage_support_wall_0.stl" scale="0.001 0.001 0.001"/>
+      </geometry>
+    </collision>
+    <collision name="storage_support_0_1">
+      <origin rpy="0 0 0" xyz="-0.169840 -0.097500 0.091000"/>
+      <geometry>
+        <mesh filename="$(arg mesh_uri)/storage_support_wall_1.stl" scale="0.001 0.001 0.001"/>
+      </geometry>
+    </collision>
+    <collision name="storage_support_0_2">
+      <origin rpy="0 0 0" xyz="-0.169840 -0.097500 0.091000"/>
+      <geometry>
+        <mesh filename="$(arg mesh_uri)/storage_support_wall_2.stl" scale="0.001 0.001 0.001"/>
+      </geometry>
+    </collision>
+    <collision name="storage_support_0_3">
+      <origin rpy="0 0 0" xyz="-0.169840 -0.097500 0.091000"/>
+      <geometry>
+        <mesh filename="$(arg mesh_uri)/storage_support_wall_3.stl" scale="0.001 0.001 0.001"/>
+      </geometry>
+    </collision>
+    <collision name="storage_support_1_0">
+      <origin rpy="0 0 0" xyz="-0.169840 -0.032500 0.091000"/>
+      <geometry>
+        <mesh filename="$(arg mesh_uri)/storage_support_wall_0.stl" scale="0.001 0.001 0.001"/>
+      </geometry>
+    </collision>
+    <collision name="storage_support_1_1">
+      <origin rpy="0 0 0" xyz="-0.169840 -0.032500 0.091000"/>
+      <geometry>
+        <mesh filename="$(arg mesh_uri)/storage_support_wall_1.stl" scale="0.001 0.001 0.001"/>
+      </geometry>
+    </collision>
+    <collision name="storage_support_1_2">
+      <origin rpy="0 0 0" xyz="-0.169840 -0.032500 0.091000"/>
+      <geometry>
+        <mesh filename="$(arg mesh_uri)/storage_support_wall_2.stl" scale="0.001 0.001 0.001"/>
+      </geometry>
+    </collision>
+    <collision name="storage_support_1_3">
+      <origin rpy="0 0 0" xyz="-0.169840 -0.032500 0.091000"/>
+      <geometry>
+        <mesh filename="$(arg mesh_uri)/storage_support_wall_3.stl" scale="0.001 0.001 0.001"/>
+      </geometry>
+    </collision>
+    <collision name="storage_support_2_0">
+      <origin rpy="0 0 0" xyz="-0.169840 0.032500 0.091000"/>
+      <geometry>
+        <mesh filename="$(arg mesh_uri)/storage_support_wall_0.stl" scale="0.001 0.001 0.001"/>
+      </geometry>
+    </collision>
+    <collision name="storage_support_2_1">
+      <origin rpy="0 0 0" xyz="-0.169840 0.032500 0.091000"/>
+      <geometry>
+        <mesh filename="$(arg mesh_uri)/storage_support_wall_1.stl" scale="0.001 0.001 0.001"/>
+      </geometry>
+    </collision>
+    <collision name="storage_support_2_2">
+      <origin rpy="0 0 0" xyz="-0.169840 0.032500 0.091000"/>
+      <geometry>
+        <mesh filename="$(arg mesh_uri)/storage_support_wall_2.stl" scale="0.001 0.001 0.001"/>
+      </geometry>
+    </collision>
+    <collision name="storage_support_2_3">
+      <origin rpy="0 0 0" xyz="-0.169840 0.032500 0.091000"/>
+      <geometry>
+        <mesh filename="$(arg mesh_uri)/storage_support_wall_3.stl" scale="0.001 0.001 0.001"/>
+      </geometry>
+    </collision>
+    <collision name="storage_support_3_0">
+      <origin rpy="0 0 0" xyz="-0.169840 0.097500 0.091000"/>
+      <geometry>
+        <mesh filename="$(arg mesh_uri)/storage_support_wall_0.stl" scale="0.001 0.001 0.001"/>
+      </geometry>
+    </collision>
+    <collision name="storage_support_3_1">
+      <origin rpy="0 0 0" xyz="-0.169840 0.097500 0.091000"/>
+      <geometry>
+        <mesh filename="$(arg mesh_uri)/storage_support_wall_1.stl" scale="0.001 0.001 0.001"/>
+      </geometry>
+    </collision>
+    <collision name="storage_support_3_2">
+      <origin rpy="0 0 0" xyz="-0.169840 0.097500 0.091000"/>
+      <geometry>
+        <mesh filename="$(arg mesh_uri)/storage_support_wall_2.stl" scale="0.001 0.001 0.001"/>
+      </geometry>
+    </collision>
+    <collision name="storage_support_3_3">
+      <origin rpy="0 0 0" xyz="-0.169840 0.097500 0.091000"/>
+      <geometry>
+        <mesh filename="$(arg mesh_uri)/storage_support_wall_3.stl" scale="0.001 0.001 0.001"/>
+      </geometry>
+    </collision>
+    <collision name="storage_support_4_0">
+      <origin rpy="0 0 0" xyz="-0.104840 -0.097500 0.091000"/>
+      <geometry>
+        <mesh filename="$(arg mesh_uri)/storage_support_wall_0.stl" scale="0.001 0.001 0.001"/>
+      </geometry>
+    </collision>
+    <collision name="storage_support_4_1">
+      <origin rpy="0 0 0" xyz="-0.104840 -0.097500 0.091000"/>
+      <geometry>
+        <mesh filename="$(arg mesh_uri)/storage_support_wall_1.stl" scale="0.001 0.001 0.001"/>
+      </geometry>
+    </collision>
+    <collision name="storage_support_4_2">
+      <origin rpy="0 0 0" xyz="-0.104840 -0.097500 0.091000"/>
+      <geometry>
+        <mesh filename="$(arg mesh_uri)/storage_support_wall_2.stl" scale="0.001 0.001 0.001"/>
+      </geometry>
+    </collision>
+    <collision name="storage_support_4_3">
+      <origin rpy="0 0 0" xyz="-0.104840 -0.097500 0.091000"/>
+      <geometry>
+        <mesh filename="$(arg mesh_uri)/storage_support_wall_3.stl" scale="0.001 0.001 0.001"/>
+      </geometry>
+    </collision>
+    <collision name="storage_support_5_0">
+      <origin rpy="0 0 0" xyz="-0.104840 -0.032500 0.091000"/>
+      <geometry>
+        <mesh filename="$(arg mesh_uri)/storage_support_wall_0.stl" scale="0.001 0.001 0.001"/>
+      </geometry>
+    </collision>
+    <collision name="storage_support_5_1">
+      <origin rpy="0 0 0" xyz="-0.104840 -0.032500 0.091000"/>
+      <geometry>
+        <mesh filename="$(arg mesh_uri)/storage_support_wall_1.stl" scale="0.001 0.001 0.001"/>
+      </geometry>
+    </collision>
+    <collision name="storage_support_5_2">
+      <origin rpy="0 0 0" xyz="-0.104840 -0.032500 0.091000"/>
+      <geometry>
+        <mesh filename="$(arg mesh_uri)/storage_support_wall_2.stl" scale="0.001 0.001 0.001"/>
+      </geometry>
+    </collision>
+    <collision name="storage_support_5_3">
+      <origin rpy="0 0 0" xyz="-0.104840 -0.032500 0.091000"/>
+      <geometry>
+        <mesh filename="$(arg mesh_uri)/storage_support_wall_3.stl" scale="0.001 0.001 0.001"/>
+      </geometry>
+    </collision>
+    <collision name="storage_support_6_0">
+      <origin rpy="0 0 0" xyz="-0.104840 0.032500 0.091000"/>
+      <geometry>
+        <mesh filename="$(arg mesh_uri)/storage_support_wall_0.stl" scale="0.001 0.001 0.001"/>
+      </geometry>
+    </collision>
+    <collision name="storage_support_6_1">
+      <origin rpy="0 0 0" xyz="-0.104840 0.032500 0.091000"/>
+      <geometry>
+        <mesh filename="$(arg mesh_uri)/storage_support_wall_1.stl" scale="0.001 0.001 0.001"/>
+      </geometry>
+    </collision>
+    <collision name="storage_support_6_2">
+      <origin rpy="0 0 0" xyz="-0.104840 0.032500 0.091000"/>
+      <geometry>
+        <mesh filename="$(arg mesh_uri)/storage_support_wall_2.stl" scale="0.001 0.001 0.001"/>
+      </geometry>
+    </collision>
+    <collision name="storage_support_6_3">
+      <origin rpy="0 0 0" xyz="-0.104840 0.032500 0.091000"/>
+      <geometry>
+        <mesh filename="$(arg mesh_uri)/storage_support_wall_3.stl" scale="0.001 0.001 0.001"/>
+      </geometry>
+    </collision>
+    <collision name="storage_support_7_0">
+      <origin rpy="0 0 0" xyz="-0.104840 0.097500 0.091000"/>
+      <geometry>
+        <mesh filename="$(arg mesh_uri)/storage_support_wall_0.stl" scale="0.001 0.001 0.001"/>
+      </geometry>
+    </collision>
+    <collision name="storage_support_7_1">
+      <origin rpy="0 0 0" xyz="-0.104840 0.097500 0.091000"/>
+      <geometry>
+        <mesh filename="$(arg mesh_uri)/storage_support_wall_1.stl" scale="0.001 0.001 0.001"/>
+      </geometry>
+    </collision>
+    <collision name="storage_support_7_2">
+      <origin rpy="0 0 0" xyz="-0.104840 0.097500 0.091000"/>
+      <geometry>
+        <mesh filename="$(arg mesh_uri)/storage_support_wall_2.stl" scale="0.001 0.001 0.001"/>
+      </geometry>
+    </collision>
+    <collision name="storage_support_7_3">
+      <origin rpy="0 0 0" xyz="-0.104840 0.097500 0.091000"/>
+      <geometry>
+        <mesh filename="$(arg mesh_uri)/storage_support_wall_3.stl" scale="0.001 0.001 0.001"/>
+      </geometry>
+    </collision>
+    <collision name="storage_support_8_0">
+      <origin rpy="0 0 0" xyz="-0.039840 -0.097500 0.091000"/>
+      <geometry>
+        <mesh filename="$(arg mesh_uri)/storage_support_wall_0.stl" scale="0.001 0.001 0.001"/>
+      </geometry>
+    </collision>
+    <collision name="storage_support_8_1">
+      <origin rpy="0 0 0" xyz="-0.039840 -0.097500 0.091000"/>
+      <geometry>
+        <mesh filename="$(arg mesh_uri)/storage_support_wall_1.stl" scale="0.001 0.001 0.001"/>
+      </geometry>
+    </collision>
+    <collision name="storage_support_8_2">
+      <origin rpy="0 0 0" xyz="-0.039840 -0.097500 0.091000"/>
+      <geometry>
+        <mesh filename="$(arg mesh_uri)/storage_support_wall_2.stl" scale="0.001 0.001 0.001"/>
+      </geometry>
+    </collision>
+    <collision name="storage_support_8_3">
+      <origin rpy="0 0 0" xyz="-0.039840 -0.097500 0.091000"/>
+      <geometry>
+        <mesh filename="$(arg mesh_uri)/storage_support_wall_3.stl" scale="0.001 0.001 0.001"/>
+      </geometry>
+    </collision>
+    <collision name="storage_support_9_0">
+      <origin rpy="0 0 0" xyz="-0.039840 -0.032500 0.091000"/>
+      <geometry>
+        <mesh filename="$(arg mesh_uri)/storage_support_wall_0.stl" scale="0.001 0.001 0.001"/>
+      </geometry>
+    </collision>
+    <collision name="storage_support_9_1">
+      <origin rpy="0 0 0" xyz="-0.039840 -0.032500 0.091000"/>
+      <geometry>
+        <mesh filename="$(arg mesh_uri)/storage_support_wall_1.stl" scale="0.001 0.001 0.001"/>
+      </geometry>
+    </collision>
+    <collision name="storage_support_9_2">
+      <origin rpy="0 0 0" xyz="-0.039840 -0.032500 0.091000"/>
+      <geometry>
+        <mesh filename="$(arg mesh_uri)/storage_support_wall_2.stl" scale="0.001 0.001 0.001"/>
+      </geometry>
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